Commit message: Adding Abductor Pollicis

File: mujoco_env/darm_hand.xml.xacro (robot description, xacro)
@@ -118,4 +118,5 @@
     <xacro:property name="flexor_superficialis_iv_origin_tf" value="-0.004 -0.013 -0.075" />
     <xacro:property name="flexor_superficialis_v_origin_tf" value="-0.012 -0.013 -0.075" />
+    <xacro:property name="abductor_pollicis_brevis_origin_tf" value="0.0223607 -0.0073321 0.0254833" />
     <!-- Tendon Origin Macro -->
     <xacro:macro name="tendon_origin" params="site_name site_tf">
@@ -178,4 +179,5 @@
                 <site name="flexor_iv_carpals_tunnel" pos="${flexor_iv_carpals_tunnel_tf}" size="${tunnel_site_size}" rgba="${tunnel_site_rgba}"/>
                 <site name="flexor_v_carpals_tunnel" pos="${flexor_v_carpals_tunnel_tf}" size="${tunnel_site_size}" rgba="${tunnel_site_rgba}"/>
+                <site name="abductor_pollicis_brevis_origin" pos="${abductor_pollicis_brevis_origin_tf}" size="${tunnel_site_size}" rgba="${tunnel_site_rgba}"/>
                 <xacro:phalanges index="ii" mcp_translation="${mcp_ii_translation}" mcp_rotation="${mcp_ii_rotation}"
                                 pp_length="${pp_ii_length}" mp_length="${mp_ii_length}" mcp_radius="${mcp_ii_radius}"

Commit message: Digit I tendon sites

File: mujoco_env/darm_hand.xml.xacro (robot description, xacro)
@@ -118,5 +118,16 @@
     <xacro:property name="flexor_superficialis_iv_origin_tf" value="-0.004 -0.013 -0.075" />
     <xacro:property name="flexor_superficialis_v_origin_tf" value="-0.012 -0.013 -0.075" />
-    <xacro:property name="abductor_pollicis_brevis_origin_tf" value="0.0223607 -0.0073321 0.0254833" />
+    <!-- Digit 1 Tendons -->
+    <xacro:property name="abductor_pollicis_brevis_carpals_tunnel_tf" value="0.0223607 -0.0073321 0.0254833" />
+    <xacro:property name="abductor_pollicis_brevis_insertion_tf" value="0.0223607 -0.0073321 0.0254833" />
+    <xacro:property name="adductor_pollicis_metacarpals_iii_tunnel_i_tf" value="0.0223607 -0.0073321 0.0254833" />
+    <xacro:property name="adductor_pollicis_metacarpals_iii_tunnel_ii_tf" value="0.0223607 -0.0073321 0.0254833" />
+    <xacro:property name="adductor_pollicis_capitate_tunnel_tf" value="0.0223607 -0.0073321 0.0254833" />
+    <xacro:property name="adductor_pollicis_insertion_tf" value="0.0223607 -0.0073321 0.0254833" />
+    <xacro:property name="flexor_pollicis_brevis_carpals_tunnel_tf" value="0.0223607 -0.0073321 0.0254833" />
+    <xacro:property name="flexor_pollicis_brevis_insertion_tf" value="0.0223607 -0.0073321 0.0254833" />
+    <xacro:property name="opponens_pollicis_carpals_tunnel_tf" value="0.0223607 -0.0073321 0.0254833" />
+    <xacro:property name="opponens_pollicis_insertion_i_tf" value="0.0223607 -0.0073321 0.0254833" />
+    <xacro:property name="opponens_pollicis_insertion_ii_tf" value="0.0223607 -0.0073321 0.0254833" />
     <!-- Tendon Origin Macro -->
     <xacro:macro name="tendon_origin" params="site_name site_tf">
@@ -179,5 +190,10 @@
                 <site name="flexor_iv_carpals_tunnel" pos="${flexor_iv_carpals_tunnel_tf}" size="${tunnel_site_size}" rgba="${tunnel_site_rgba}"/>
                 <site name="flexor_v_carpals_tunnel" pos="${flexor_v_carpals_tunnel_tf}" size="${tunnel_site_size}" rgba="${tunnel_site_rgba}"/>
-                <site name="abductor_pollicis_brevis_origin" pos="${abductor_pollicis_brevis_origin_tf}" size="${tunnel_site_size}" rgba="${tunnel_site_rgba}"/>
+                <site name="abductor_pollicis_brevis_carpals_tunnel" pos="${abductor_pollicis_brevis_carpals_tunnel_tf}" size="${tunnel_site_size}" rgba="${tunnel_site_rgba}"/>
+                <site name="adductor_pollicis_metacarpals_iii_tunnel_i" pos="${adductor_pollicis_metacarpals_iii_tunnel_i_tf}" size="${tunnel_site_size}" rgba="${tunnel_site_rgba}"/>
+                <site name="adductor_pollicis_metacarpals_iii_tunnel_ii" pos="${adductor_pollicis_metacarpals_iii_tunnel_ii_tf}" size="${tunnel_site_size}" rgba="${tunnel_site_rgba}"/>
+                <site name="adductor_pollicis_capitate_tunnel" pos="${adductor_pollicis_capitate_tunnel_tf}" size="${tunnel_site_size}" rgba="${tunnel_site_rgba}"/>
+                <site name="flexor_pollicis_brevis_carpals_tunnel" pos="${flexor_pollicis_brevis_carpals_tunnel_tf}" size="${tunnel_site_size}" rgba="${tunnel_site_rgba}"/>
+                <site name="opponens_pollicis_carpals_tunnel" pos="${opponens_pollicis_carpals_tunnel_tf}" size="${tunnel_site_size}" rgba="${tunnel_site_rgba}"/>
                 <xacro:phalanges index="ii" mcp_translation="${mcp_ii_translation}" mcp_rotation="${mcp_ii_rotation}"
                                 pp_length="${pp_ii_length}" mp_length="${mp_ii_length}" mcp_radius="${mcp_ii_radius}"
@@ -224,5 +240,10 @@
                 <xacro:phalanx_i index="i" cm_translation="${cm_i_translation}" cm_rotation="${cm_i_rotation}"
                                 centre_block_offset="${cm_i_centre_block_offset}" metacarpal_length="${metacarpal_i_length}"
-                                pp_length="${pp_i_length}" />
+                                pp_length="${pp_i_length}"
+                                abductor_pollicis_brevis_insertion_tf="${abductor_pollicis_brevis_insertion_tf}"
+                                adductor_pollicis_insertion_tf="${adductor_pollicis_insertion_tf}"
+                                flexor_pollicis_brevis_insertion_tf="${flexor_pollicis_brevis_insertion_tf}"
+                                opponens_pollicis_insertion_i_tf="${opponens_pollicis_insertion_i_tf}"
+                                opponens_pollicis_insertion_ii_tf="${opponens_pollicis_insertion_ii_tf}" />
                 </body>
         </body>

File: mujoco_env/phalanges.xml.xacro (robot description, xacro)
@@ -77,5 +77,7 @@
         </body>
     </xacro:macro>
-    <xacro:macro name="phalanx_i" params="index cm_translation cm_rotation centre_block_offset metacarpal_length pp_length">
+    <xacro:macro name="phalanx_i" params="index cm_translation cm_rotation centre_block_offset metacarpal_length
+        pp_length abductor_pollicis_brevis_insertion_tf adductor_pollicis_insertion_tf flexor_pollicis_brevis_insertion_tf
+        opponens_pollicis_insertion_i_tf opponens_pollicis_insertion_ii_tf">
         <body name="proximal_cm_i_centre_block" pos="${cm_translation}" euler="${cm_rotation}">
             <joint type="hinge" axis="1 0 0" />
@@ -85,9 +87,14 @@
                 <geom type="mesh" mesh="distal_cm_i_centre_block_mesh" />
                 <body name="metacarpal_i" pos="0 0 0" euler="0 0 0">
-                  <joint type="hinge" axis="0 1 0" pos="0 0 0" />
-                  <geom type="mesh" mesh="metacarpal_i_mesh" />
+                    <joint type="hinge" axis="0 1 0" pos="0 0 0" />
+                    <geom type="mesh" mesh="metacarpal_i_mesh" />
+                    <site name="opponens_pollicis_insertion_i" pos="${opponens_pollicis_insertion_i_tf}" size="${tunnel_site_size}" rgba="${tunnel_site_rgba}"/>
+                    <site name="opponens_pollicis_insertion_ii" pos="${opponens_pollicis_insertion_ii_tf}" size="${tunnel_site_size}" rgba="${tunnel_site_rgba}"/>
                         <body name="proximal_phalanx_${index}" pos="0 0 ${metacarpal_length}" euler="0 0 0">
                             <joint type="hinge" axis="1 0 0" />
                             <geom type="mesh" mesh="proximal_phalanx_${index}_mesh" rgba="1 0 0 1" />
+                            <site name="abductor_pollicis_brevis_insertion" pos="${abductor_pollicis_brevis_insertion_tf}" size="${tunnel_site_size}" rgba="${tunnel_site_rgba}"/>
+                            <site name="adductor_pollicis_insertion" pos="${adductor_pollicis_insertion_tf}" size="${tunnel_site_size}" rgba="${tunnel_site_rgba}"/>
+                            <site name="flexor_pollicis_brevis_insertion" pos="${flexor_pollicis_brevis_insertion_tf}" size="${tunnel_site_size}" rgba="${tunnel_site_rgba}"/>
                             <body name="distal_phalanx_${index}" pos="0 0 ${pp_length}" euler="0 0 0">
                                 <joint type="hinge" axis="1 0 0" />

Commit message: Digit I tendon sites tf parameter

File: mujoco_env/darm_hand.xml.xacro (robot description, xacro)
@@ -119,15 +119,15 @@
     <xacro:property name="flexor_superficialis_v_origin_tf" value="-0.012 -0.013 -0.075" />
     <!-- Digit 1 Tendons -->
-    <xacro:property name="abductor_pollicis_brevis_carpals_tunnel_tf" value="0.0223607 -0.0073321 0.0254833" />
-    <xacro:property name="abductor_pollicis_brevis_insertion_tf" value="0.0223607 -0.0073321 0.0254833" />
-    <xacro:property name="adductor_pollicis_metacarpals_iii_tunnel_i_tf" value="0.0223607 -0.0073321 0.0254833" />
-    <xacro:property name="adductor_pollicis_metacarpals_iii_tunnel_ii_tf" value="0.0223607 -0.0073321 0.0254833" />
-    <xacro:property name="adductor_pollicis_capitate_tunnel_tf" value="0.0223607 -0.0073321 0.0254833" />
-    <xacro:property name="adductor_pollicis_insertion_tf" value="0.0223607 -0.0073321 0.0254833" />
-    <xacro:property name="flexor_pollicis_brevis_carpals_tunnel_tf" value="0.0223607 -0.0073321 0.0254833" />
-    <xacro:property name="flexor_pollicis_brevis_insertion_tf" value="0.0223607 -0.0073321 0.0254833" />
-    <xacro:property name="opponens_pollicis_carpals_tunnel_tf" value="0.0223607 -0.0073321 0.0254833" />
-    <xacro:property name="opponens_pollicis_insertion_i_tf" value="0.0223607 -0.0073321 0.0254833" />
-    <xacro:property name="opponens_pollicis_insertion_ii_tf" value="0.0223607 -0.0073321 0.0254833" />
+    <xacro:property name="abductor_pollicis_brevis_carpals_tunnel_tf" value="0.024963 -0.016395 0.022153" />
+    <xacro:property name="abductor_pollicis_brevis_insertion_tf" value="0.008 0.0 0.0" />
+    <xacro:property name="adductor_pollicis_metacarpals_iii_tunnel_i_tf" value="0.009064 -0.000907 0.041" />
+    <xacro:property name="adductor_pollicis_metacarpals_iii_tunnel_ii_tf" value="0.012845 0.001949 0.07707" />
+    <xacro:property name="adductor_pollicis_capitate_tunnel_tf" value="-0.001286 -0.010 0.016" />
+    <xacro:property name="adductor_pollicis_insertion_tf" value="-0.008 0.0 0.0" />
+    <xacro:property name="flexor_pollicis_brevis_carpals_tunnel_tf" value="0.0128 -0.00957 0.020" />
+    <xacro:property name="flexor_pollicis_brevis_insertion_tf" value="0.005 -0.005598 0.008406" />
+    <xacro:property name="opponens_pollicis_carpals_tunnel_tf" value="0.0128 -0.00957 0.020" />
+    <xacro:property name="opponens_pollicis_insertion_i_tf" value="0.0055 0.0048 0.009875" />
+    <xacro:property name="opponens_pollicis_insertion_ii_tf" value="0.00543 0.005595 0.03379" />
     <!-- Tendon Origin Macro -->
     <xacro:macro name="tendon_origin" params="site_name site_tf">

Commit message: Thumb Tendons

File: mujoco_env/darm_hand.xml.xacro (robot description, xacro)
@@ -7,9 +7,13 @@
     <xacro:property name="rc_joint_length" value="0.0235" />
     <!-- Digit I -->
-    <xacro:property name="cm_i_translation" value="0.0223607 -0.0073321 0.0254833" />
+    <xacro:property name="cm_i_translation" value="${[0.0223607, -0.0073321, 0.0254833]}" />
     <xacro:property name="cm_i_rotation" value="24 -15 -75" />
-    <xacro:property name="cm_i_centre_block_offset" value="0 0 0.013" />
+    <xacro:property name="cm_i_centre_block_offset" value="${[0, 0, 0.013]}" />
     <xacro:property name="metacarpal_i_length" value="0.0395" />
     <xacro:property name="pp_i_length" value="0.0335" />
+    <xacro:property name="proximal_cm_i_radius" value="0.0085" />
+    <xacro:property name="distal_cm_i_radius" value="0.0075" />
+    <xacro:property name="mcp_i_radius" value="0.0075" />
+    <xacro:property name="ip_i_radius" value="0.0065" />
     <!-- Digit II -->
     <xacro:property name="mcp_ii_translation" value="0.0293 0.0087 0.0908" />
@@ -196,4 +200,6 @@
                 <site name="flexor_pollicis_brevis_carpals_tunnel" pos="${flexor_pollicis_brevis_carpals_tunnel_tf}" size="${tunnel_site_size}" rgba="${tunnel_site_rgba}"/>
                 <site name="opponens_pollicis_carpals_tunnel" pos="${opponens_pollicis_carpals_tunnel_tf}" size="${tunnel_site_size}" rgba="${tunnel_site_rgba}"/>
+                <site name="proximal_cm_i_wrap_dorsal_sidesite" pos="${cm_i_translation[0]+1.2*proximal_cm_i_radius+sidesite_size} ${cm_i_translation[1]} ${cm_i_translation[2]}" size="${sidesite_size}" rgba="${sidesite_rgba}" />
+                <site name="proximal_cm_i_wrap_palmar_sidesite" pos="${cm_i_translation[0]-1.2*proximal_cm_i_radius-sidesite_size} ${cm_i_translation[1]} ${cm_i_translation[2]}" size="${sidesite_size}" rgba="${sidesite_rgba}" />
                 <xacro:phalanges index="ii" mcp_translation="${mcp_ii_translation}" mcp_rotation="${mcp_ii_rotation}"
                                 pp_length="${pp_ii_length}" mp_length="${mp_ii_length}" mcp_radius="${mcp_ii_radius}"
@@ -240,5 +246,6 @@
                 <xacro:phalanx_i index="i" cm_translation="${cm_i_translation}" cm_rotation="${cm_i_rotation}"
                                 centre_block_offset="${cm_i_centre_block_offset}" metacarpal_length="${metacarpal_i_length}"
-                                pp_length="${pp_i_length}"
+                                pp_length="${pp_i_length}" proximal_cm_radius="${proximal_cm_i_radius}"
+                                distal_cm_radius="${distal_cm_i_radius}" mcp_radius="${mcp_i_radius}" ip_radius="${ip_i_radius}"
                                 abductor_pollicis_brevis_insertion_tf="${abductor_pollicis_brevis_insertion_tf}"
                                 adductor_pollicis_insertion_tf="${adductor_pollicis_insertion_tf}"

File: mujoco_env/phalanges.xml.xacro (robot description, xacro)
@@ -61,6 +61,6 @@
                     <joint type="hinge" axis="0 1 0" pos="0 0 -${metacarpal_length}" />
                     <geom type="mesh" mesh="metacarpal_v_mesh" />
-                    <site name="flexor_v_metacarpals_tunnel" pos="0 0.009 -${metacarpal_length}" size="${tunnel_site_size}" rgba="${tunnel_site_rgba}"/>
-                    <site name="extensor_communis_v_metacarpals_tunnel" pos="0 -0.009 -${metacarpal_length}" size="${tunnel_site_size}" rgba="${tunnel_site_rgba}"/>
+                    <site name="flexor_v_metacarpals_tunnel" pos="0 -0.009 -${metacarpal_length}" size="${tunnel_site_size}" rgba="${tunnel_site_rgba}"/>
+                    <site name="extensor_communis_v_metacarpals_tunnel" pos="0 0.009 -${metacarpal_length}" size="${tunnel_site_size}" rgba="${tunnel_site_rgba}"/>
                     <xacro:phalanges index="${index}" mcp_translation="${mcp_translation}" mcp_rotation="${mcp_rotation}"
                                     pp_length="${pp_length}" mp_length="${mp_length}" mcp_radius="${mcp_radius}"
@@ -78,23 +78,34 @@
     </xacro:macro>
     <xacro:macro name="phalanx_i" params="index cm_translation cm_rotation centre_block_offset metacarpal_length
-        pp_length abductor_pollicis_brevis_insertion_tf adductor_pollicis_insertion_tf flexor_pollicis_brevis_insertion_tf
-        opponens_pollicis_insertion_i_tf opponens_pollicis_insertion_ii_tf">
-        <body name="proximal_cm_i_centre_block" pos="${cm_translation}" euler="${cm_rotation}">
+        pp_length proximal_cm_radius distal_cm_radius mcp_radius ip_radius abductor_pollicis_brevis_insertion_tf adductor_pollicis_insertion_tf flexor_pollicis_brevis_insertion_tf
+        opponens_pollicis_insertion_i_tf opponens_pollicis_insertion_ii_tf
+        wrap_rgba:='0 0 1 0.2'">
+        <body name="proximal_cm_i_centre_block" pos="${cm_translation[0]} ${cm_translation[1]} ${cm_translation[2]}" euler="${cm_rotation}">
             <joint type="hinge" axis="1 0 0" />
             <geom type="mesh" mesh="proximal_cm_i_centre_block_mesh" />
-            <body name="distal_cm_i_centre_block" pos="${centre_block_offset}" euler="0 0 0">
+            <geom name="proximal_cm_i_wrap" type="cylinder" size="${proximal_cm_radius} 0.010" euler="0 90 0" rgba="${wrap_rgba}" />
+            <site name="distal_cm_${index}_wrap_dorsal_sidesite" pos="${distal_cm_radius+sidesite_size} 0 ${centre_block_offset[2]}" size="${sidesite_size}" rgba="${sidesite_rgba}" />
+            <site name="distal_cm_${index}_wrap_palmar_sidesite" pos="-${distal_cm_radius+sidesite_size} 0 ${centre_block_offset[2]}" size="${sidesite_size}" rgba="${sidesite_rgba}" />
+            <body name="distal_cm_i_centre_block" pos="${centre_block_offset[0]} ${centre_block_offset[1]} ${centre_block_offset[2]}" euler="0 0 0">
                 <joint type="hinge" axis="0 0 1" />
                 <geom type="mesh" mesh="distal_cm_i_centre_block_mesh" />
+                <geom name="distal_cm_i_wrap" type="cylinder" size="${distal_cm_radius} 0.009" euler="90 0 0" rgba="${wrap_rgba}" />
                 <body name="metacarpal_i" pos="0 0 0" euler="0 0 0">
                     <joint type="hinge" axis="0 1 0" pos="0 0 0" />
                     <geom type="mesh" mesh="metacarpal_i_mesh" />
+                    <geom name="mcp_i_wrap" type="cylinder" pos="0 0 ${metacarpal_length}" size="${mcp_radius} 0.008" euler="0 90 0" rgba="${wrap_rgba}" />
                     <site name="opponens_pollicis_insertion_i" pos="${opponens_pollicis_insertion_i_tf}" size="${tunnel_site_size}" rgba="${tunnel_site_rgba}"/>
                     <site name="opponens_pollicis_insertion_ii" pos="${opponens_pollicis_insertion_ii_tf}" size="${tunnel_site_size}" rgba="${tunnel_site_rgba}"/>
+                    <site name="mcp_${index}_wrap_dorsal_sidesite" pos="0 ${mcp_radius+sidesite_size} ${metacarpal_length}" size="${sidesite_size}" rgba="${sidesite_rgba}" />
+                    <site name="mcp_${index}_wrap_palmar_sidesite" pos="0 -${mcp_radius+sidesite_size} ${metacarpal_length}" size="${sidesite_size}" rgba="${sidesite_rgba}" />
                         <body name="proximal_phalanx_${index}" pos="0 0 ${metacarpal_length}" euler="0 0 0">
                             <joint type="hinge" axis="1 0 0" />
                             <geom type="mesh" mesh="proximal_phalanx_${index}_mesh" rgba="1 0 0 1" />
+                            <geom name="ip_i_wrap" type="cylinder" pos="0 0 ${pp_length}" size="${ip_radius} 0.008" euler="0 90 0" rgba="${wrap_rgba}" />
                             <site name="abductor_pollicis_brevis_insertion" pos="${abductor_pollicis_brevis_insertion_tf}" size="${tunnel_site_size}" rgba="${tunnel_site_rgba}"/>
                             <site name="adductor_pollicis_insertion" pos="${adductor_pollicis_insertion_tf}" size="${tunnel_site_size}" rgba="${tunnel_site_rgba}"/>
                             <site name="flexor_pollicis_brevis_insertion" pos="${flexor_pollicis_brevis_insertion_tf}" size="${tunnel_site_size}" rgba="${tunnel_site_rgba}"/>
+                            <site name="ip_${index}_wrap_dorsal_sidesite" pos="0 ${ip_radius+sidesite_size} ${pp_length}" size="${sidesite_size}" rgba="${sidesite_rgba}" />
+                            <site name="ip_${index}_wrap_palmar_sidesite" pos="0 -${ip_radius+sidesite_size} ${pp_length}" size="${sidesite_size}" rgba="${sidesite_rgba}" />
                             <body name="distal_phalanx_${index}" pos="0 0 ${pp_length}" euler="0 0 0">
                                 <joint type="hinge" axis="1 0 0" />

File: mujoco_env/tendon.xml.xacro (robot description, xacro)
@@ -70,3 +70,29 @@
     <xacro:phalanges_tendons index="iv" />
     <xacro:phalanges_tendons index="v" />
+    <spatial name="abductor_pollicis_brevis" width="0.0004">
+        <site site="abductor_pollicis_brevis_carpals_tunnel" />
+        <geom geom="distal_cm_i_wrap" sidesite="distal_cm_i_wrap_dorsal_sidesite" />
+        <site site="abductor_pollicis_brevis_insertion" />
+    </spatial>
+    <spatial name="adductor_pollicis_oblique" width="0.0004">
+        <site site="adductor_pollicis_capitate_tunnel" />
+        <geom geom="proximal_cm_i_wrap" sidesite="proximal_cm_i_wrap_palmar_sidesite" />
+        <site site="adductor_pollicis_insertion" />
+    </spatial>
+    <spatial name="adductor_pollicis_transverse" width="0.0004">
+        <site site="adductor_pollicis_metacarpals_iii_tunnel_i" />
+        <site site="adductor_pollicis_metacarpals_iii_tunnel_ii" />
+        <site site="adductor_pollicis_insertion" />
+    </spatial>
+    <spatial name="flexor_pollicis_brevis" width="0.0004">
+        <site site="flexor_pollicis_brevis_carpals_tunnel" />
+        <geom geom="distal_cm_i_wrap" sidesite="distal_cm_i_wrap_dorsal_sidesite" />
+        <site site="flexor_pollicis_brevis_insertion" />
+    </spatial>
+    <spatial name="opponens_pollicis" width="0.0004">
+        <site site="opponens_pollicis_carpals_tunnel" />
+        <geom geom="distal_cm_i_wrap" sidesite="distal_cm_i_wrap_dorsal_sidesite" />
+        <site site="opponens_pollicis_insertion_i" />
+        <site site="opponens_pollicis_insertion_ii" />
+    </spatial>
 </tendon>
