Commit message: Digit I and V Tendons

File: mujoco_env/darm_hand.xml.xacro (robot description, xacro)
@@ -134,4 +134,11 @@
     <xacro:property name="opponens_pollicis_insertion_i_tf" value="0.0055 0.0048 0.009875" />
     <xacro:property name="opponens_pollicis_insertion_ii_tf" value="0.00543 0.005595 0.03379" />
+    <xacro:property name="flexor_pollicis_longus_insertion_tf" value="0.0 -0.005 0.007" />
+    <xacro:property name="flexor_pollicis_longus_origin_tf" value="-0.012 -0.013 -0.075" />
+    <xacro:property name="extensor_pollicis_brevis_insertion_tf" value="0.0 0.006 0.008" />
+    <xacro:property name="extensor_pollicis_brevis_origin_tf" value="0.012 0.013 -0.035" />
+    <xacro:property name="extensor_pollicis_longus_insertion_tf" value="0.0 0.005 0.007" />
+    <xacro:property name="extensor_pollicis_longus_origin_tf" value="0.012 0.013 -0.035" />
+    <xacro:property name="abductor_pollicis_longus_origin_tf" value="0.012 0.013 -0.035" />
     <!-- Tendon Origin Macro -->
     <xacro:macro name="tendon_origin" params="site_name site_tf">
@@ -168,4 +175,8 @@
         <xacro:tendon_origin site_name="dorsal_interossei_iv_origin" site_tf="${dorsal_interossei_iv_origin_tf}" />
         <xacro:tendon_origin site_name="dorsal_interossei_v_origin" site_tf="${dorsal_interossei_v_origin_tf}" />
+        <xacro:tendon_origin site_name="flexor_pollicis_longus_origin" site_tf="${flexor_pollicis_longus_origin_tf}" />
+        <xacro:tendon_origin site_name="extensor_pollicis_brevis_origin" site_tf="${extensor_pollicis_brevis_origin_tf}" />
+        <xacro:tendon_origin site_name="extensor_pollicis_longus_origin" site_tf="${extensor_pollicis_longus_origin_tf}" />
+        <xacro:tendon_origin site_name="abductor_pollicis_longus_origin" site_tf="${abductor_pollicis_longus_origin_tf}" />
         <!-- TODO: Measure this accurately from f360 -->
         <body name="rc_centre_block" pos="${rc_joint_tf[0]} ${rc_joint_tf[1]} ${rc_joint_tf[2]}" euler="0 0 0">
@@ -252,5 +263,8 @@
                                 flexor_pollicis_brevis_insertion_tf="${flexor_pollicis_brevis_insertion_tf}"
                                 opponens_pollicis_insertion_i_tf="${opponens_pollicis_insertion_i_tf}"
-                                opponens_pollicis_insertion_ii_tf="${opponens_pollicis_insertion_ii_tf}" />
+                                opponens_pollicis_insertion_ii_tf="${opponens_pollicis_insertion_ii_tf}"
+                                flexor_pollicis_longus_insertion_tf="${flexor_pollicis_longus_insertion_tf}"
+                                extensor_pollicis_brevis_insertion_tf="${extensor_pollicis_brevis_insertion_tf}"
+                                extensor_pollicis_longus_insertion_tf="${extensor_pollicis_longus_insertion_tf}" />
                 </body>
         </body>

File: mujoco_env/phalanges.xml.xacro (robot description, xacro)
@@ -79,5 +79,6 @@
     <xacro:macro name="phalanx_i" params="index cm_translation cm_rotation centre_block_offset metacarpal_length
         pp_length proximal_cm_radius distal_cm_radius mcp_radius ip_radius abductor_pollicis_brevis_insertion_tf adductor_pollicis_insertion_tf flexor_pollicis_brevis_insertion_tf
-        opponens_pollicis_insertion_i_tf opponens_pollicis_insertion_ii_tf
+        opponens_pollicis_insertion_i_tf opponens_pollicis_insertion_ii_tf flexor_pollicis_longus_insertion_tf
+        extensor_pollicis_brevis_insertion_tf extensor_pollicis_longus_insertion_tf
         wrap_rgba:='0 0 1 0.2'">
         <body name="proximal_cm_i_centre_block" pos="${cm_translation[0]} ${cm_translation[1]} ${cm_translation[2]}" euler="${cm_rotation}">
@@ -106,4 +107,5 @@
                             <site name="adductor_pollicis_insertion" pos="${adductor_pollicis_insertion_tf}" size="${tunnel_site_size}" rgba="${tunnel_site_rgba}"/>
                             <site name="flexor_pollicis_brevis_insertion" pos="${flexor_pollicis_brevis_insertion_tf}" size="${tunnel_site_size}" rgba="${tunnel_site_rgba}"/>
+                            <site name="extensor_pollicis_brevis_insertion" pos="${extensor_pollicis_brevis_insertion_tf}" size="${site_size}" rgba="${site_rgba}"/>
                             <site name="ip_${index}_wrap_dorsal_sidesite" pos="0 ${ip_radius+sidesite_size} ${pp_length}" size="${sidesite_size}" rgba="${sidesite_rgba}" />
                             <site name="ip_${index}_wrap_palmar_sidesite" pos="0 -${ip_radius+sidesite_size} ${pp_length}" size="${sidesite_size}" rgba="${sidesite_rgba}" />
@@ -111,4 +113,6 @@
                                 <joint type="hinge" axis="1 0 0" />
                                 <geom type="mesh" mesh="distal_phalanx_${index}_mesh" rgba="0 0 1 1" />
+                                <site name="flexor_pollicis_longus_insertion" pos="${flexor_pollicis_longus_insertion_tf}" size="${site_size}" rgba="${site_rgba}"/>
+                                <site name="extensor_pollicis_longus_insertion" pos="${extensor_pollicis_longus_insertion_tf}" size="${site_size}" rgba="${site_rgba}"/>
                             </body>
                         </body>

Commit message: Added all Joints Limits

File: mujoco_env/darm_hand.xml.xacro (robot description, xacro)
@@ -118,13 +118,13 @@
     <xacro:property name="dorsal_interossei_iv_origin_tf" value="-0.003 -0.013 -0.055" />
     <xacro:property name="dorsal_interossei_v_origin_tf" value="-0.010 -0.013 -0.055" />
-    <xacro:property name="flexor_superficialis_ii_origin_tf" value="0.012 -0.013 -0.075" />
-    <xacro:property name="flexor_superficialis_iii_origin_tf" value="0.004 -0.013 -0.075" />
-    <xacro:property name="flexor_superficialis_iv_origin_tf" value="-0.004 -0.013 -0.075" />
-    <xacro:property name="flexor_superficialis_v_origin_tf" value="-0.012 -0.013 -0.075" />
+    <xacro:property name="flexor_superficialis_ii_origin_tf" value="0.012 -0.013 -0.065" />
+    <xacro:property name="flexor_superficialis_iii_origin_tf" value="0.004 -0.013 -0.065" />
+    <xacro:property name="flexor_superficialis_iv_origin_tf" value="-0.004 -0.013 -0.065" />
+    <xacro:property name="flexor_superficialis_v_origin_tf" value="-0.012 -0.013 -0.065" />
     <!-- Digit 1 Tendons -->
     <xacro:property name="abductor_pollicis_brevis_carpals_tunnel_tf" value="0.024963 -0.016395 0.022153" />
     <xacro:property name="abductor_pollicis_brevis_insertion_tf" value="0.008 0.0 0.0" />
     <xacro:property name="adductor_pollicis_metacarpals_iii_tunnel_i_tf" value="0.009064 -0.000907 0.041" />
-    <xacro:property name="adductor_pollicis_metacarpals_iii_tunnel_ii_tf" value="0.012845 0.001949 0.07707" />
+    <xacro:property name="adductor_pollicis_metacarpals_iii_tunnel_ii_tf" value="0.011 0.001949 0.070" />
     <xacro:property name="adductor_pollicis_capitate_tunnel_tf" value="-0.001286 -0.010 0.016" />
     <xacro:property name="adductor_pollicis_insertion_tf" value="-0.008 0.0 0.0" />
@@ -135,13 +135,29 @@
     <xacro:property name="opponens_pollicis_insertion_ii_tf" value="0.00543 0.005595 0.03379" />
     <xacro:property name="flexor_pollicis_longus_insertion_tf" value="0.0 -0.005 0.007" />
-    <xacro:property name="flexor_pollicis_longus_origin_tf" value="-0.012 -0.013 -0.075" />
+    <xacro:property name="flexor_pollicis_longus_origin_tf" value="0.012 -0.013 -0.075" />
     <xacro:property name="extensor_pollicis_brevis_insertion_tf" value="0.0 0.006 0.008" />
-    <xacro:property name="extensor_pollicis_brevis_origin_tf" value="0.012 0.013 -0.035" />
+    <xacro:property name="extensor_pollicis_brevis_origin_tf" value="0.012 0.013 -0.045" />
     <xacro:property name="extensor_pollicis_longus_insertion_tf" value="0.0 0.005 0.007" />
-    <xacro:property name="extensor_pollicis_longus_origin_tf" value="0.012 0.013 -0.035" />
-    <xacro:property name="abductor_pollicis_longus_origin_tf" value="0.012 0.013 -0.035" />
+    <xacro:property name="extensor_pollicis_longus_origin_tf" value="0.004 0.013 -0.045" />
+    <xacro:property name="abductor_pollicis_longus_origin_tf" value="0.012 0.013 -0.055" />
+    <!-- Digit V Tendons -->
+    <xacro:property name="opponens_digiti_minimi_origin_tf" value="-0.012 -0.013 -0.075" />
+    <xacro:property name="opponens_digiti_minimi_carpals_tunnel_tf" value="-0.004421 -0.010 0.016" />
+    <xacro:property name="opponens_digiti_minimi_insertion_i_tf" value="-0.0065 0.005506 -0.026175" />
+    <xacro:property name="opponens_digiti_minimi_insertion_ii_tf" value="-0.0045 0.00665 -0.013738" />
+    <!-- Carpal Tendons -->
+    <xacro:property name="flexor_carpi_radialis_insertion_tf" value="0.02 -0.015 0.016" />
+    <xacro:property name="flexor_carpi_ulnaris_insertion_tf" value="-0.0185 -0.012 0.016" />
+    <xacro:property name="extensor_carpi_radialis_insertion_tf" value="0.021 0.01 0.016" />
+    <xacro:property name="extensor_carpi_ulnaris_insertion_tf" value="-0.0185 0.012 0.016" />
+    <xacro:property name="flexor_carpi_radialis_origin_tf" value="0.012 -0.013 -0.085" />
+    <xacro:property name="flexor_carpi_ulnaris_origin_tf" value="-0.012 -0.013 -0.085" />
+    <xacro:property name="extensor_carpi_radialis_origin_tf" value="0.012 0.013 -0.065" />
+    <xacro:property name="extensor_carpi_ulnaris_origin_tf" value="-0.012 0.013 -0.065" />
     <!-- Tendon Origin Macro -->
     <xacro:macro name="tendon_origin" params="site_name site_tf">
         <body>
+            <geom type="sphere" size="${.5*origin_site_size}" />
+            <joint name="${site_name}_joint" type="slide" axis="0 0 1" pos="${site_tf}" />
             <site name="${site_name}" pos="${site_tf}" size="${origin_site_size}" rgba="${origin_site_rgba}"/>
         </body>
@@ -149,5 +165,5 @@
     <body name="forearm" pos="0 0 0.12" euler="0 0 0" childclass="darm_meshes">
         <geom type="mesh" mesh="forearm_mesh" />
-        <geom name="rc_joint_wrap" type="cylinder" pos="${rc_joint_tf[0]} ${rc_joint_tf[1]} ${rc_joint_tf[2]}"
+        <geom class="wrap_geom" name="rc_joint_wrap" type="cylinder" pos="${rc_joint_tf[0]} ${rc_joint_tf[1]} ${rc_joint_tf[2]}"
             size="${rc_joint_radius} ${rc_joint_length}" euler="0 90 0" rgba="${wrap_rgba}" />
         <site name="rc_joint_wrap_dorsal_sidesite" pos="0 ${rc_joint_radius+sidesite_size} ${rc_joint_tf[2]}"
@@ -155,4 +171,8 @@
         <site name="rc_joint_wrap_palmar_sidesite" pos="0 -${rc_joint_radius+sidesite_size} ${rc_joint_tf[2]}"
             size="${sidesite_size}" rgba="${sidesite_rgba}" />
+        <xacro:tendon_origin site_name="flexor_carpi_radialis_origin" site_tf="${flexor_carpi_radialis_origin_tf}" />
+        <xacro:tendon_origin site_name="flexor_carpi_ulnaris_origin" site_tf="${flexor_carpi_ulnaris_origin_tf}" />
+        <xacro:tendon_origin site_name="extensor_carpi_radialis_origin" site_tf="${extensor_carpi_radialis_origin_tf}" />
+        <xacro:tendon_origin site_name="extensor_carpi_ulnaris_origin" site_tf="${extensor_carpi_ulnaris_origin_tf}" />
         <xacro:tendon_origin site_name="extensor_communis_ii_origin" site_tf="${extensor_communis_ii_origin_tf}" />
         <xacro:tendon_origin site_name="extensor_communis_iii_origin" site_tf="${extensor_communis_iii_origin_tf}" />
@@ -179,9 +199,19 @@
         <xacro:tendon_origin site_name="extensor_pollicis_longus_origin" site_tf="${extensor_pollicis_longus_origin_tf}" />
         <xacro:tendon_origin site_name="abductor_pollicis_longus_origin" site_tf="${abductor_pollicis_longus_origin_tf}" />
+        <xacro:tendon_origin site_name="opponens_digiti_minimi_origin" site_tf="${opponens_digiti_minimi_origin_tf}" />
         <!-- TODO: Measure this accurately from f360 -->
         <body name="rc_centre_block" pos="${rc_joint_tf[0]} ${rc_joint_tf[1]} ${rc_joint_tf[2]}" euler="0 0 0">
+            <!-- <joint type="hinge" axis="0 1 0" pos="0 0 -0.032" limited="true" range="-20 10" /> -->
             <geom type="mesh" mesh="rc_centre_block_mesh" />
             <body name="carpals_metacarpals" pos="0 0 0" euler="0 0 0">
+                <joint type="hinge" axis="1 0 0" limited="true" range="-90 90" />
                 <geom type="mesh" mesh="carpals_metacarpals_mesh" />
+                <geom class="wrap_geom" pos="${mcp_ii_translation}" name="mcp_ii_wrap" type="cylinder" size="${mcp_ii_radius} ${mcp_ii_radius}" euler="0 90 0" rgba="${wrap_rgba}" />
+                <geom class="wrap_geom" pos="${mcp_iii_translation}" name="mcp_iii_wrap" type="cylinder" size="${mcp_iii_radius} ${mcp_iii_radius}" euler="0 90 0" rgba="${wrap_rgba}" />
+                <geom class="wrap_geom" pos="${mcp_iv_translation}" name="mcp_iv_wrap" type="cylinder" size="${mcp_iv_radius} ${mcp_iv_radius}" euler="0 90 0" rgba="${wrap_rgba}" />
+                <site name="flexor_carpi_radialis_insertion" pos="${flexor_carpi_radialis_insertion_tf}" size="${tunnel_site_size}" rgba="${tunnel_site_rgba}"/>
+                <site name="flexor_carpi_ulnaris_insertion" pos="${flexor_carpi_ulnaris_insertion_tf}" size="${tunnel_site_size}" rgba="${tunnel_site_rgba}"/>
+                <site name="extensor_carpi_radialis_insertion" pos="${extensor_carpi_radialis_insertion_tf}" size="${tunnel_site_size}" rgba="${tunnel_site_rgba}"/>
+                <site name="extensor_carpi_ulnaris_insertion" pos="${extensor_carpi_ulnaris_insertion_tf}" size="${tunnel_site_size}" rgba="${tunnel_site_rgba}"/>
                 <site name="extensor_communis_ii_carpals_tunnel" pos="${extensor_communis_ii_carpals_tunnel_tf}"
                     size="${tunnel_site_size}" rgba="${tunnel_site_rgba}"/>
@@ -213,4 +243,5 @@
                 <site name="proximal_cm_i_wrap_dorsal_sidesite" pos="${cm_i_translation[0]+1.2*proximal_cm_i_radius+sidesite_size} ${cm_i_translation[1]} ${cm_i_translation[2]}" size="${sidesite_size}" rgba="${sidesite_rgba}" />
                 <site name="proximal_cm_i_wrap_palmar_sidesite" pos="${cm_i_translation[0]-1.2*proximal_cm_i_radius-sidesite_size} ${cm_i_translation[1]} ${cm_i_translation[2]}" size="${sidesite_size}" rgba="${sidesite_rgba}" />
+                <site name="opponens_digiti_minimi_carpals_tunnel" pos="${opponens_digiti_minimi_carpals_tunnel_tf}" size="${tunnel_site_size}" rgba="${tunnel_site_rgba}" />
                 <xacro:phalanges index="ii" mcp_translation="${mcp_ii_translation}" mcp_rotation="${mcp_ii_rotation}"
                                 pp_length="${pp_ii_length}" mp_length="${mp_ii_length}" mcp_radius="${mcp_ii_radius}"
@@ -243,16 +274,4 @@
                                 flexor_profundus_insertion_tf="${flexor_profundus_iv_insertion_tf}"
                                 dp_extensor_hood_insertion_tf="${dp_iv_extensor_hood_insertion_tf}" />
-                <xacro:phalanx_v index="v" cm_translation="${cm_v_translation}" cm_rotation="${cm_v_rotation}"
-                                centre_block_offset="${cm_v_centre_block_offset}" metacarpal_length="${metacarpal_v_length}"
-                                mcp_translation="${mcp_v_translation}" mcp_rotation="${mcp_v_rotation}" pp_length="${pp_v_length}"
-                                mp_length="${mp_v_length}" mcp_radius="${mcp_v_radius}"
-                                pip_radius="${pip_v_radius}" dip_radius="${dip_v_radius}"
-                                dorsal_interossei_insertion_tf="${dorsal_interossei_v_insertion_tf}"
-                                palmar_interossei_insertion_tf="${palmar_interossei_v_insertion_tf}"
-                                pp_extensor_communis_insertion_tf="${pp_v_extensor_communis_insertion_tf}"
-                                flexor_superficialis_insertion_tf="${flexor_superficialis_v_insertion_tf}"
-                                mp_extensor_hood_insertion_tf="${mp_v_extensor_hood_insertion_tf}"
-                                flexor_profundus_insertion_tf="${flexor_profundus_v_insertion_tf}"
-                                dp_extensor_hood_insertion_tf="${dp_v_extensor_hood_insertion_tf}" />
                 <xacro:phalanx_i index="i" cm_translation="${cm_i_translation}" cm_rotation="${cm_i_rotation}"
                                 centre_block_offset="${cm_i_centre_block_offset}" metacarpal_length="${metacarpal_i_length}"
@@ -267,5 +286,19 @@
                                 extensor_pollicis_brevis_insertion_tf="${extensor_pollicis_brevis_insertion_tf}"
                                 extensor_pollicis_longus_insertion_tf="${extensor_pollicis_longus_insertion_tf}" />
-                </body>
+                <xacro:phalanx_v index="v" cm_translation="${cm_v_translation}" cm_rotation="${cm_v_rotation}"
+                                centre_block_offset="${cm_v_centre_block_offset}" metacarpal_length="${metacarpal_v_length}"
+                                mcp_translation="${mcp_v_translation}" mcp_rotation="${mcp_v_rotation}" pp_length="${pp_v_length}"
+                                mp_length="${mp_v_length}" mcp_radius="${mcp_v_radius}"
+                                pip_radius="${pip_v_radius}" dip_radius="${dip_v_radius}"
+                                dorsal_interossei_insertion_tf="${dorsal_interossei_v_insertion_tf}"
+                                palmar_interossei_insertion_tf="${palmar_interossei_v_insertion_tf}"
+                                pp_extensor_communis_insertion_tf="${pp_v_extensor_communis_insertion_tf}"
+                                flexor_superficialis_insertion_tf="${flexor_superficialis_v_insertion_tf}"
+                                mp_extensor_hood_insertion_tf="${mp_v_extensor_hood_insertion_tf}"
+                                flexor_profundus_insertion_tf="${flexor_profundus_v_insertion_tf}"
+                                dp_extensor_hood_insertion_tf="${dp_v_extensor_hood_insertion_tf}"
+                                opponens_digiti_minimi_insertion_i_tf="${opponens_digiti_minimi_insertion_i_tf}"
+                                opponens_digiti_minimi_insertion_ii_tf="${opponens_digiti_minimi_insertion_ii_tf}" />
+            </body>
         </body>
     </body>
