Commit message: Completed adding all tendons

File: mujoco_env/darm_hand.xml.xacro (robot description, xacro)
@@ -70,4 +70,6 @@
     <xacro:property name="pp_v_length" value="0.0416" />
     <xacro:property name="mp_v_length" value="0.0247" />
+    <xacro:property name="proximal_cm_v_radius" value="0.007" />
+    <xacro:property name="distal_cm_v_radius" value="0.007" />
     <xacro:property name="mcp_v_radius" value="0.0095" />
     <xacro:property name="pip_v_radius" value="0.0060" />
@@ -123,27 +125,39 @@
     <xacro:property name="flexor_superficialis_v_origin_tf" value="-0.012 -0.013 -0.065" />
     <!-- Digit 1 Tendons -->
+    <xacro:property name="abductor_pollicis_brevis_origin_tf" value="0.012 -0.013 -0.075" />
     <xacro:property name="abductor_pollicis_brevis_carpals_tunnel_tf" value="0.024963 -0.016395 0.022153" />
     <xacro:property name="abductor_pollicis_brevis_insertion_tf" value="0.008 0.0 0.0" />
+    <xacro:property name="adductor_pollicis_origin_tf" value="0.0 -0.013 -0.085" />
     <xacro:property name="adductor_pollicis_metacarpals_iii_tunnel_i_tf" value="0.009064 -0.000907 0.041" />
     <xacro:property name="adductor_pollicis_metacarpals_iii_tunnel_ii_tf" value="0.011 0.001949 0.070" />
-    <xacro:property name="adductor_pollicis_capitate_tunnel_tf" value="-0.001286 -0.010 0.016" />
+    <xacro:property name="adductor_pollicis_capitate_tunnel_tf" value="0.0 -0.010 0.016" />
     <xacro:property name="adductor_pollicis_insertion_tf" value="-0.008 0.0 0.0" />
+    <xacro:property name="flexor_pollicis_brevis_origin_tf" value="0.004 -0.013 -0.075" />
     <xacro:property name="flexor_pollicis_brevis_carpals_tunnel_tf" value="0.0128 -0.00957 0.020" />
     <xacro:property name="flexor_pollicis_brevis_insertion_tf" value="0.005 -0.005598 0.008406" />
+    <xacro:property name="opponens_pollicis_origin_tf" value="0.0 -0.013 -0.075" />
     <xacro:property name="opponens_pollicis_carpals_tunnel_tf" value="0.0128 -0.00957 0.020" />
     <xacro:property name="opponens_pollicis_insertion_i_tf" value="0.0055 0.0048 0.009875" />
     <xacro:property name="opponens_pollicis_insertion_ii_tf" value="0.00543 0.005595 0.03379" />
+    <xacro:property name="flexor_pollicis_longus_origin_tf" value="0.008 -0.013 -0.075" />
     <xacro:property name="flexor_pollicis_longus_insertion_tf" value="0.0 -0.005 0.007" />
-    <xacro:property name="flexor_pollicis_longus_origin_tf" value="0.012 -0.013 -0.075" />
     <xacro:property name="extensor_pollicis_brevis_insertion_tf" value="0.0 0.006 0.008" />
     <xacro:property name="extensor_pollicis_brevis_origin_tf" value="0.012 0.013 -0.045" />
     <xacro:property name="extensor_pollicis_longus_insertion_tf" value="0.0 0.005 0.007" />
     <xacro:property name="extensor_pollicis_longus_origin_tf" value="0.004 0.013 -0.045" />
+    <!-- brevis and longus tunnel -->
+    <xacro:property name="extensor_pollicis_carpals_tunnel_tf" value="0.024 0.001 0.016" />
     <xacro:property name="abductor_pollicis_longus_origin_tf" value="0.012 0.013 -0.055" />
+    <xacro:property name="abductor_pollicis_longus_insertion_tf" value="0.0055 0.0 0.008" />
+    <xacro:property name="metacarpal_i_flexor_tunnel_tf" value="0.0 -0.0065 ${metacarpal_i_length/2}" />
+    <xacro:property name="metacarpal_i_extensor_tunnel_tf" value="0.0 0.0065 ${metacarpal_i_length/2}" />
+    <xacro:property name="pp_i_flexor_tunnel_tf" value="0.0 -0.005 ${pp_i_length/2}" />
+    <xacro:property name="pp_i_extensor_tunnel_tf" value="0.0 0.005 ${pp_i_length/2}" />
     <!-- Digit V Tendons -->
     <xacro:property name="opponens_digiti_minimi_origin_tf" value="-0.012 -0.013 -0.075" />
-    <xacro:property name="opponens_digiti_minimi_carpals_tunnel_tf" value="-0.004421 -0.010 0.016" />
+    <xacro:property name="opponens_digiti_minimi_carpals_tunnel_tf" value="-0.007 -0.010 0.016" />
     <xacro:property name="opponens_digiti_minimi_insertion_i_tf" value="-0.0065 0.005506 -0.026175" />
     <xacro:property name="opponens_digiti_minimi_insertion_ii_tf" value="-0.0045 0.00665 -0.013738" />
+    <xacro:property name="opponens_digiti_minimi_distal_cm_v_tunnel_tf" value="-0.0065 -0.0035 -0.007" />
     <!-- Carpal Tendons -->
     <xacro:property name="flexor_carpi_radialis_insertion_tf" value="0.02 -0.015 0.016" />
@@ -165,6 +179,4 @@
     <body name="forearm" pos="0 0 0.12" euler="0 0 0" childclass="darm_meshes">
         <geom type="mesh" mesh="forearm_mesh" />
-        <geom class="wrap_geom" name="rc_joint_wrap" type="cylinder" pos="${rc_joint_tf[0]} ${rc_joint_tf[1]} ${rc_joint_tf[2]}"
-            size="${rc_joint_radius} ${rc_joint_length}" euler="0 90 0" rgba="${wrap_rgba}" />
         <site name="rc_joint_wrap_dorsal_sidesite" pos="0 ${rc_joint_radius+sidesite_size} ${rc_joint_tf[2]}"
             size="${sidesite_size}" rgba="${sidesite_rgba}" />
@@ -196,12 +208,18 @@
         <xacro:tendon_origin site_name="dorsal_interossei_v_origin" site_tf="${dorsal_interossei_v_origin_tf}" />
         <xacro:tendon_origin site_name="flexor_pollicis_longus_origin" site_tf="${flexor_pollicis_longus_origin_tf}" />
+        <xacro:tendon_origin site_name="flexor_pollicis_brevis_origin" site_tf="${flexor_pollicis_brevis_origin_tf}" />
         <xacro:tendon_origin site_name="extensor_pollicis_brevis_origin" site_tf="${extensor_pollicis_brevis_origin_tf}" />
         <xacro:tendon_origin site_name="extensor_pollicis_longus_origin" site_tf="${extensor_pollicis_longus_origin_tf}" />
         <xacro:tendon_origin site_name="abductor_pollicis_longus_origin" site_tf="${abductor_pollicis_longus_origin_tf}" />
+        <xacro:tendon_origin site_name="abductor_pollicis_brevis_origin" site_tf="${abductor_pollicis_brevis_origin_tf}" />
+        <xacro:tendon_origin site_name="opponens_pollicis_origin" site_tf="${opponens_pollicis_origin_tf}" />
+        <xacro:tendon_origin site_name="adductor_pollicis_origin" site_tf="${adductor_pollicis_origin_tf}" />
         <xacro:tendon_origin site_name="opponens_digiti_minimi_origin" site_tf="${opponens_digiti_minimi_origin_tf}" />
         <!-- TODO: Measure this accurately from f360 -->
         <body name="rc_centre_block" pos="${rc_joint_tf[0]} ${rc_joint_tf[1]} ${rc_joint_tf[2]}" euler="0 0 0">
-            <!-- <joint type="hinge" axis="0 1 0" pos="0 0 -0.032" limited="true" range="-20 10" /> -->
+            <joint type="hinge" axis="0 1 0" pos="0 0 -0.032" limited="true" range="-20 10" />
             <geom type="mesh" mesh="rc_centre_block_mesh" />
+            <geom class="wrap_geom" name="rc_joint_wrap" type="cylinder"
+                size="${rc_joint_radius} ${rc_joint_length}" euler="0 90 0" rgba="${wrap_rgba}" />
             <body name="carpals_metacarpals" pos="0 0 0" euler="0 0 0">
                 <joint type="hinge" axis="1 0 0" limited="true" range="-90 90" />
@@ -214,4 +232,5 @@
                 <site name="extensor_carpi_radialis_insertion" pos="${extensor_carpi_radialis_insertion_tf}" size="${tunnel_site_size}" rgba="${tunnel_site_rgba}"/>
                 <site name="extensor_carpi_ulnaris_insertion" pos="${extensor_carpi_ulnaris_insertion_tf}" size="${tunnel_site_size}" rgba="${tunnel_site_rgba}"/>
+                <site name="extensor_pollicis_carpals_tunnel" pos="${extensor_pollicis_carpals_tunnel_tf}" size="${tunnel_site_size}" rgba="${tunnel_site_rgba}"/>
                 <site name="extensor_communis_ii_carpals_tunnel" pos="${extensor_communis_ii_carpals_tunnel_tf}"
                     size="${tunnel_site_size}" rgba="${tunnel_site_rgba}"/>
@@ -279,4 +298,5 @@
                                 distal_cm_radius="${distal_cm_i_radius}" mcp_radius="${mcp_i_radius}" ip_radius="${ip_i_radius}"
                                 abductor_pollicis_brevis_insertion_tf="${abductor_pollicis_brevis_insertion_tf}"
+                                abductor_pollicis_longus_insertion_tf="${abductor_pollicis_longus_insertion_tf}"
                                 adductor_pollicis_insertion_tf="${adductor_pollicis_insertion_tf}"
                                 flexor_pollicis_brevis_insertion_tf="${flexor_pollicis_brevis_insertion_tf}"
@@ -285,9 +305,14 @@
                                 flexor_pollicis_longus_insertion_tf="${flexor_pollicis_longus_insertion_tf}"
                                 extensor_pollicis_brevis_insertion_tf="${extensor_pollicis_brevis_insertion_tf}"
-                                extensor_pollicis_longus_insertion_tf="${extensor_pollicis_longus_insertion_tf}" />
+                                extensor_pollicis_longus_insertion_tf="${extensor_pollicis_longus_insertion_tf}"
+                                metacarpal_i_flexor_tunnel_tf="${metacarpal_i_flexor_tunnel_tf}"
+                                metacarpal_i_extensor_tunnel_tf="${metacarpal_i_extensor_tunnel_tf}"
+                                pp_i_flexor_tunnel_tf="${pp_i_flexor_tunnel_tf}"
+                                pp_i_extensor_tunnel_tf="${pp_i_extensor_tunnel_tf}" />
                 <xacro:phalanx_v index="v" cm_translation="${cm_v_translation}" cm_rotation="${cm_v_rotation}"
                                 centre_block_offset="${cm_v_centre_block_offset}" metacarpal_length="${metacarpal_v_length}"
                                 mcp_translation="${mcp_v_translation}" mcp_rotation="${mcp_v_rotation}" pp_length="${pp_v_length}"
-                                mp_length="${mp_v_length}" mcp_radius="${mcp_v_radius}"
+                                mp_length="${mp_v_length}" proximal_cm_radius="${proximal_cm_v_radius}"
+                                distal_cm_radius="${distal_cm_v_radius}" mcp_radius="${mcp_v_radius}"
                                 pip_radius="${pip_v_radius}" dip_radius="${dip_v_radius}"
                                 dorsal_interossei_insertion_tf="${dorsal_interossei_v_insertion_tf}"
@@ -299,5 +324,6 @@
                                 dp_extensor_hood_insertion_tf="${dp_v_extensor_hood_insertion_tf}"
                                 opponens_digiti_minimi_insertion_i_tf="${opponens_digiti_minimi_insertion_i_tf}"
-                                opponens_digiti_minimi_insertion_ii_tf="${opponens_digiti_minimi_insertion_ii_tf}" />
+                                opponens_digiti_minimi_insertion_ii_tf="${opponens_digiti_minimi_insertion_ii_tf}"
+                                opponens_digiti_minimi_distal_cm_v_tunnel_tf="${opponens_digiti_minimi_distal_cm_v_tunnel_tf}" />
             </body>
         </body>

File: mujoco_env/phalanges.xml.xacro (robot description, xacro)
@@ -47,16 +47,24 @@
     </xacro:macro>
     <xacro:macro name="phalanx_v" params="index cm_translation cm_rotation centre_block_offset metacarpal_length mcp_translation
-        mcp_rotation pp_length mp_length mcp_radius pip_radius dip_radius dorsal_interossei_insertion_tf
+        mcp_rotation pp_length mp_length proximal_cm_radius distal_cm_radius mcp_radius pip_radius dip_radius dorsal_interossei_insertion_tf
         palmar_interossei_insertion_tf pp_extensor_communis_insertion_tf flexor_superficialis_insertion_tf
         mp_extensor_hood_insertion_tf flexor_profundus_insertion_tf dp_extensor_hood_insertion_tf
         opponens_digiti_minimi_insertion_i_tf opponens_digiti_minimi_insertion_ii_tf
-        tunnelsite_size:=0.0015 tunnelsite_rgba:='0.5 0.5 0.5 1'
-        site_size:=0.002 site_rgba:='0.1 0.1 0.1 1'">
+        opponens_digiti_minimi_distal_cm_v_tunnel_tf
+        tunnelsite_size:=0.0015 tunnelsite_rgba:='0.5 0.5 0.5 1' sidesite_rgba:='1 1 1 0.2'
+        sidesite_size:=0.001 site_size:=0.002 site_rgba:='0.1 0.1 0.1 1'">
         <body name="proximal_cm_v_centre_block" pos="${cm_translation}" euler="${cm_rotation}">
             <joint type="hinge" axis="1 0 0" limited="true" range="-10 10" />
             <geom type="mesh" mesh="proximal_cm_v_centre_block_mesh" />
+            <geom class="wrap_geom" name="proximal_cm_v_wrap" type="cylinder" size="${proximal_cm_radius} 0.009" euler="0 90 0" rgba="${wrap_rgba}" />
+            <site name="proximal_cm_v_wrap_dorsal_sidesite" pos="0 ${proximal_cm_radius+sidesite_size} 0" size="${sidesite_size}" rgba="${sidesite_rgba}" />
+            <site name="proximal_cm_v_wrap_palmar_sidesite" pos="0 -${proximal_cm_radius+sidesite_size} 0" size="${sidesite_size}" rgba="${sidesite_rgba}" />
             <body name="distal_cm_v_centre_block" pos="${centre_block_offset}" euler="0 0 0">
                 <joint type="hinge" axis="0 0 1" limited="true" range="-10 10" />
                 <geom type="mesh" mesh="distal_cm_v_centre_block_mesh" />
+                <geom class="wrap_geom" name="distal_cm_v_wrap" type="cylinder" size="${distal_cm_radius} 0.008" euler="90 0 0" rgba="${wrap_rgba}" />
+                <site name="distal_cm_v_wrap_ulnar_sidesite" pos="-${distal_cm_radius+sidesite_size} 0 0" size="${sidesite_size}" rgba="${sidesite_rgba}" />
+                <site name="distal_cm_v_wrap_radial_sidesite" pos="${distal_cm_radius+sidesite_size} 0 0" size="${sidesite_size}" rgba="${sidesite_rgba}" />
+                <site name="opponens_digiti_minimi_distal_cm_v_tunnel" pos="${opponens_digiti_minimi_distal_cm_v_tunnel_tf}" size="${tunnel_site_size}" rgba="${tunnel_site_rgba}"/>
                 <body name="metacarpal_v" pos="0 0 ${metacarpal_length}" euler="0 0 0">
                     <joint type="hinge" axis="0 1 0" pos="0 0 -${metacarpal_length}"  limited="true" range="-5 5" />
@@ -82,9 +90,12 @@
     </xacro:macro>
     <xacro:macro name="phalanx_i" params="index cm_translation cm_rotation centre_block_offset metacarpal_length
-        pp_length proximal_cm_radius distal_cm_radius mcp_radius ip_radius abductor_pollicis_brevis_insertion_tf adductor_pollicis_insertion_tf flexor_pollicis_brevis_insertion_tf
+        pp_length proximal_cm_radius distal_cm_radius mcp_radius ip_radius abductor_pollicis_brevis_insertion_tf
+        abductor_pollicis_longus_insertion_tf adductor_pollicis_insertion_tf flexor_pollicis_brevis_insertion_tf
         opponens_pollicis_insertion_i_tf opponens_pollicis_insertion_ii_tf flexor_pollicis_longus_insertion_tf
         extensor_pollicis_brevis_insertion_tf extensor_pollicis_longus_insertion_tf
+        metacarpal_i_flexor_tunnel_tf pp_i_flexor_tunnel_tf metacarpal_i_extensor_tunnel_tf pp_i_extensor_tunnel_tf
         wrap_rgba:='0 0 1 0.2' pp_rgba:='1 0 0 1' dp_rgba:='0 0 1 1'
-        site_size:=0.002 site_rgba:='0.1 0.1 0.1 1'">
+        site_size:=0.002 site_rgba:='0.1 0.1 0.1 1'
+        tunnelsite_size:=0.0015 tunnelsite_rgba:='0.5 0.5 0.5 1' sidesite_rgba:='1 1 1 0.2' ">
         <body name="proximal_cm_i_centre_block" pos="${cm_translation[0]} ${cm_translation[1]} ${cm_translation[2]}" euler="${cm_rotation}">
             <joint type="hinge" axis="1 0 0" limited="true" range="-50 -10" />
@@ -103,10 +114,15 @@
                     <site name="opponens_pollicis_insertion_i" pos="${opponens_pollicis_insertion_i_tf}" size="${tunnel_site_size}" rgba="${tunnel_site_rgba}"/>
                     <site name="opponens_pollicis_insertion_ii" pos="${opponens_pollicis_insertion_ii_tf}" size="${tunnel_site_size}" rgba="${tunnel_site_rgba}"/>
+                    <site name="abductor_pollicis_longus_insertion" pos="${abductor_pollicis_longus_insertion_tf}" size="${tunnel_site_size}" rgba="${tunnel_site_rgba}"/>
                     <site name="mcp_${index}_wrap_dorsal_sidesite" pos="0 ${mcp_radius+sidesite_size} ${metacarpal_length}" size="${sidesite_size}" rgba="${sidesite_rgba}" />
                     <site name="mcp_${index}_wrap_palmar_sidesite" pos="0 -${mcp_radius+sidesite_size} ${metacarpal_length}" size="${sidesite_size}" rgba="${sidesite_rgba}" />
+                    <site name="metacarpal_i_flexor_tunnel" pos="${metacarpal_i_flexor_tunnel_tf}" size="${tunnel_site_size}" rgba="${tunnel_site_rgba}"/>
+                    <site name="metacarpal_i_extensor_tunnel" pos="${metacarpal_i_extensor_tunnel_tf}" size="${tunnel_site_size}" rgba="${tunnel_site_rgba}"/>
                         <body name="proximal_phalanx_${index}" pos="0 0 ${metacarpal_length}" euler="0 0 0">
                             <joint type="hinge" axis="1 0 0" limited="true" range="-10 90" />
                             <geom type="mesh" mesh="proximal_phalanx_${index}_mesh" rgba="${pp_rgba}" />
                             <geom class="wrap_geom" name="ip_i_wrap" type="cylinder" pos="0 0 ${pp_length}" size="${ip_radius} 0.008" euler="0 90 0" rgba="${wrap_rgba}" />
+                            <site name="pp_i_flexor_tunnel" pos="${pp_i_flexor_tunnel_tf}" size="${tunnel_site_size}" rgba="${pp_rgba}"/>
+                            <site name="pp_i_extensor_tunnel" pos="${pp_i_extensor_tunnel_tf}" size="${tunnel_site_size}" rgba="${pp_rgba}"/>
                             <site name="abductor_pollicis_brevis_insertion" pos="${abductor_pollicis_brevis_insertion_tf}" size="${tunnel_site_size}" rgba="${tunnel_site_rgba}"/>
                             <site name="adductor_pollicis_insertion" pos="${adductor_pollicis_insertion_tf}" size="${tunnel_site_size}" rgba="${tunnel_site_rgba}"/>
