Commit message: Completed adding all tendons

File: mujoco_env/tendon.xml.xacro (robot description, xacro)
@@ -1,4 +1,6 @@
 <?xml version="1.0" encoding="UTF-8"?>
 <tendon xmlns:xacro="http://wiki.ros.org/xacro">
+    <!-- TODO: Interossei Position on Metacarpals -->
+    <!-- TODO: Muscles with three fibres -->
     <xacro:macro name="phalanges_tendons" params="index">
         <spatial name="dorsal_interossei_${index}" width="0.0004">
@@ -50,5 +52,5 @@
             <site site="pp_${index}_flexor_tunnel" />
             <geom geom="pip_${index}_wrap" sidesite="pip_${index}_wrap_palmar_sidesite" />
-            <site site="flexor_superficialis_${index}_insertion" />
+            <!-- <site site="flexor_superficialis_${index}_insertion" /> -->
             <site site="mp_${index}_flexor_tunnel" />
             <geom geom="dip_${index}_wrap" sidesite="dip_${index}_wrap_palmar_sidesite" />
@@ -72,17 +74,21 @@
     <!-- Pollicis Muscles -->
     <spatial name="abductor_pollicis_brevis" width="0.0004">
-        <!-- Combined with the longus tendon -->
-        <site site="abductor_pollicis_longus_origin" />
+        <site site="abductor_pollicis_brevis_origin" />
+        <geom geom="rc_joint_wrap" sidesite="rc_joint_wrap_palmar_sidesite" />
         <site site="abductor_pollicis_brevis_carpals_tunnel" />
-        <!-- TODO: Add insertion at the base of metacarpal one | not carpals -->
         <geom geom="distal_cm_i_wrap" sidesite="distal_cm_i_wrap_dorsal_sidesite" />
         <site site="abductor_pollicis_brevis_insertion" />
     </spatial>
     <spatial name="adductor_pollicis_oblique" width="0.0004">
+        <site site="adductor_pollicis_origin" />
+        <geom geom="rc_joint_wrap" sidesite="rc_joint_wrap_palmar_sidesite" />
         <site site="adductor_pollicis_capitate_tunnel" />
-        <geom geom="proximal_cm_i_wrap" sidesite="proximal_cm_i_wrap_palmar_sidesite" />
+        <geom geom="distal_cm_i_wrap" sidesite="proximal_cm_i_wrap_palmar_sidesite" />
         <site site="adductor_pollicis_insertion" />
     </spatial>
     <spatial name="adductor_pollicis_transverse" width="0.0004">
+        <site site="adductor_pollicis_origin" />
+        <geom geom="rc_joint_wrap" sidesite="rc_joint_wrap_palmar_sidesite" />
+        <site site="adductor_pollicis_capitate_tunnel" />
         <site site="adductor_pollicis_metacarpals_iii_tunnel_i" />
         <site site="adductor_pollicis_metacarpals_iii_tunnel_ii" />
@@ -90,4 +96,6 @@
     </spatial>
     <spatial name="flexor_pollicis_brevis" width="0.0004">
+        <site site="flexor_pollicis_brevis_origin" />
+        <geom geom="rc_joint_wrap" sidesite="rc_joint_wrap_palmar_sidesite" />
         <site site="flexor_pollicis_brevis_carpals_tunnel" />
         <geom geom="distal_cm_i_wrap" sidesite="distal_cm_i_wrap_dorsal_sidesite" />
@@ -95,4 +103,6 @@
     </spatial>
     <spatial name="opponens_pollicis" width="0.0004">
+        <site site="opponens_pollicis_origin" />
+        <geom geom="rc_joint_wrap" sidesite="rc_joint_wrap_palmar_sidesite" />
         <site site="opponens_pollicis_carpals_tunnel" />
         <geom geom="distal_cm_i_wrap" sidesite="distal_cm_i_wrap_dorsal_sidesite" />
@@ -102,41 +112,70 @@
     <spatial name="flexor_pollicis_longus" width="0.0004">
         <site site="flexor_pollicis_longus_origin" />
+        <geom geom="rc_joint_wrap" sidesite="rc_joint_wrap_palmar_sidesite" />
+        <site site="flexor_pollicis_brevis_carpals_tunnel" />
+        <geom geom="proximal_cm_i_wrap" sidesite="proximal_cm_i_wrap_palmar_sidesite" />
+        <site site="metacarpal_i_flexor_tunnel" />
+        <geom geom="mcp_i_wrap" sidesite="mcp_i_wrap_palmar_sidesite" />
+        <site site="pp_i_flexor_tunnel" />
+        <geom geom="ip_i_wrap" sidesite="ip_i_wrap_palmar_sidesite" />
         <site site="flexor_pollicis_longus_insertion" />
     </spatial>
     <spatial name="extensor_pollicis_brevis" width="0.0004">
         <site site="extensor_pollicis_brevis_origin" />
+        <geom geom="rc_joint_wrap" sidesite="rc_joint_wrap_dorsal_sidesite" />
+        <site site="extensor_pollicis_carpals_tunnel" />
+        <geom geom="proximal_cm_i_wrap" sidesite="proximal_cm_i_wrap_dorsal_sidesite" />
+        <site site="metacarpal_i_extensor_tunnel" />
+        <geom geom="mcp_i_wrap" sidesite="mcp_i_wrap_dorsal_sidesite" />
         <site site="extensor_pollicis_brevis_insertion" />
     </spatial>
     <spatial name="extensor_pollicis_longus" width="0.0004">
         <site site="extensor_pollicis_longus_origin" />
+        <geom geom="rc_joint_wrap" sidesite="rc_joint_wrap_dorsal_sidesite" />
+        <site site="extensor_pollicis_carpals_tunnel" />
+        <geom geom="proximal_cm_i_wrap" sidesite="proximal_cm_i_wrap_dorsal_sidesite" />
+        <site site="metacarpal_i_extensor_tunnel" />
+        <geom geom="mcp_i_wrap" sidesite="mcp_i_wrap_dorsal_sidesite" />
+        <site site="pp_i_extensor_tunnel" />
+        <geom geom="ip_i_wrap" sidesite="ip_i_wrap_dorsal_sidesite" />
         <site site="extensor_pollicis_longus_insertion" />
     </spatial>
-    <!-- Combines with abductor pollicis brevis
     <spatial name="abductor_pollicis_longus" width="0.0004">
         <site site="abductor_pollicis_longus_origin" />
-        <site site="abductor_pollicis_brevis_carpals_tunnel" />
-    </spatial> -->
+        <geom geom="rc_joint_wrap" sidesite="rc_joint_wrap_dorsal_sidesite" />
+        <site site="extensor_pollicis_carpals_tunnel" />
+        <geom geom="distal_cm_i_wrap" sidesite="distal_cm_i_wrap_dorsal_sidesite" />
+        <site site="abductor_pollicis_longus_insertion" />
+    </spatial>
     <!-- Digiti Minimi -->
     <spatial name="opponens_digiti_minimi" width="0.0004">
         <site site="opponens_digiti_minimi_origin" />
+        <geom geom="rc_joint_wrap" sidesite="rc_joint_wrap_palmar_sidesite" />
         <site site="opponens_digiti_minimi_carpals_tunnel" />
+        <geom geom="proximal_cm_v_wrap" sidesite="proximal_cm_v_wrap_palmar_sidesite" />
+        <site site="opponens_digiti_minimi_distal_cm_v_tunnel" />
+        <geom geom="distal_cm_v_wrap" sidesite="distal_cm_v_wrap_ulnar_sidesite" />
         <site site="opponens_digiti_minimi_insertion_i" />
         <site site="opponens_digiti_minimi_insertion_ii" />
     </spatial>
     <!-- Carpals, RC Joint -->
-    <spatial name="flexor_carpi_radialis" width="0.0004">
+    <spatial name="flexor_carpi_radialis" width="0.0004" limited="true" range="0 0.07">
         <site site="flexor_carpi_radialis_origin" />
+        <geom geom="rc_joint_wrap" sidesite="rc_joint_wrap_palmar_sidesite" />
         <site site="flexor_carpi_radialis_insertion" />
     </spatial>
-    <spatial name="flexor_carpi_ulnaris" width="0.0004">
+    <spatial name="flexor_carpi_ulnaris" width="0.0004" limited="true" range="0 0.07">
         <site site="flexor_carpi_ulnaris_origin" />
+        <geom geom="rc_joint_wrap" sidesite="rc_joint_wrap_palmar_sidesite" />
         <site site="flexor_carpi_ulnaris_insertion" />
     </spatial>
     <spatial name="extensor_carpi_radialis" width="0.0004">
         <site site="extensor_carpi_radialis_origin" />
+        <geom geom="rc_joint_wrap" sidesite="rc_joint_wrap_dorsal_sidesite" />
         <site site="extensor_carpi_radialis_insertion" />
     </spatial>
     <spatial name="extensor_carpi_ulnaris" width="0.0004">
         <site site="extensor_carpi_ulnaris_origin" />
+        <geom geom="rc_joint_wrap" sidesite="rc_joint_wrap_dorsal_sidesite" />
         <site site="extensor_carpi_ulnaris_insertion" />
     </spatial>

Commit message: Actuators added to tendons

File: mujoco_env/darm_hand.xml.xacro (robot description, xacro)
@@ -171,9 +171,9 @@
     <!-- Tendon Origin Macro -->
     <xacro:macro name="tendon_origin" params="site_name site_tf">
-        <body>
-            <geom type="sphere" size="${.5*origin_site_size}" />
-            <joint name="${site_name}_joint" type="slide" axis="0 0 1" pos="${site_tf}" />
-            <site name="${site_name}" pos="${site_tf}" size="${origin_site_size}" rgba="${origin_site_rgba}"/>
-        </body>
+        <site name="${site_name}" pos="${site_tf}" size="${origin_site_size}" rgba="${origin_site_rgba}"/>
+        <!-- <body> -->
+            <!-- <geom type="sphere" size="${.5*origin_site_size}" /> -->
+            <!-- <joint name="${site_name}_joint" type="slide" axis="0 0 1" pos="${site_tf}" /> -->
+        <!-- </body> -->
     </xacro:macro>
     <body name="forearm" pos="0 0 0.12" euler="0 0 0" childclass="darm_meshes">

File: mujoco_env/tendon.xml.xacro (robot description, xacro)
@@ -160,10 +160,10 @@
     </spatial>
     <!-- Carpals, RC Joint -->
-    <spatial name="flexor_carpi_radialis" width="0.0004" limited="true" range="0 0.07">
+    <spatial name="flexor_carpi_radialis" width="0.0004">
         <site site="flexor_carpi_radialis_origin" />
         <geom geom="rc_joint_wrap" sidesite="rc_joint_wrap_palmar_sidesite" />
         <site site="flexor_carpi_radialis_insertion" />
     </spatial>
-    <spatial name="flexor_carpi_ulnaris" width="0.0004" limited="true" range="0 0.07">
+    <spatial name="flexor_carpi_ulnaris" width="0.0004">
         <site site="flexor_carpi_ulnaris_origin" />
         <geom geom="rc_joint_wrap" sidesite="rc_joint_wrap_palmar_sidesite" />

Commit message: Added Fingertip Sites

File: mujoco_env/darm_hand.xml.xacro (robot description, xacro)
@@ -12,4 +12,6 @@
     <xacro:property name="metacarpal_i_length" value="0.0395" />
     <xacro:property name="pp_i_length" value="0.0335" />
+    <!-- <xacro:property name="dp_i_length" value="0.0294" /> -->
+    <xacro:property name="dp_i_length" value="0.027" />
     <xacro:property name="proximal_cm_i_radius" value="0.0085" />
     <xacro:property name="distal_cm_i_radius" value="0.0075" />
@@ -21,4 +23,5 @@
     <xacro:property name="pp_ii_length" value="0.0488" />
     <xacro:property name="mp_ii_length" value="0.0268" />
+    <xacro:property name="dp_ii_length" value="0.0211" />
     <xacro:property name="mcp_ii_radius" value="0.0110" />
     <xacro:property name="pip_ii_radius" value="0.0065" />
@@ -36,4 +39,5 @@
     <xacro:property name="pp_iii_length" value="0.0520" />
     <xacro:property name="mp_iii_length" value="0.0335" />
+    <xacro:property name="dp_iii_length" value="0.0204" />
     <xacro:property name="mcp_iii_radius" value="0.0110" />
     <xacro:property name="pip_iii_radius" value="0.0070" />
@@ -51,4 +55,5 @@
     <xacro:property name="pp_iv_length" value="0.0487" />
     <xacro:property name="mp_iv_length" value="0.0330" />
+    <xacro:property name="dp_iv_length" value="0.0202" />
     <xacro:property name="mcp_iv_radius" value="0.0095" />
     <xacro:property name="pip_iv_radius" value="0.0065" />
@@ -70,4 +75,5 @@
     <xacro:property name="pp_v_length" value="0.0416" />
     <xacro:property name="mp_v_length" value="0.0247" />
+    <xacro:property name="dp_v_length" value="0.0185" />
     <xacro:property name="proximal_cm_v_radius" value="0.007" />
     <xacro:property name="distal_cm_v_radius" value="0.007" />
@@ -268,5 +274,6 @@
                 <site name="opponens_digiti_minimi_carpals_tunnel" pos="${opponens_digiti_minimi_carpals_tunnel_tf}" size="${tunnel_site_size}" rgba="${tunnel_site_rgba}" />
                 <xacro:phalanges index="ii" mcp_translation="${mcp_ii_translation}" mcp_rotation="${mcp_ii_rotation}"
-                                pp_length="${pp_ii_length}" mp_length="${mp_ii_length}" mcp_radius="${mcp_ii_radius}"
+                                pp_length="${pp_ii_length}" mp_length="${mp_ii_length}" dp_length="${dp_ii_length}"
+                                mcp_radius="${mcp_ii_radius}"
                                 pip_radius="${pip_ii_radius}" dip_radius="${dip_ii_radius}"
                                 dorsal_interossei_insertion_tf="${dorsal_interossei_ii_insertion_tf}"
@@ -278,5 +285,6 @@
                                 dp_extensor_hood_insertion_tf="${dp_ii_extensor_hood_insertion_tf}" />
                 <xacro:phalanges index="iii" mcp_translation="${mcp_iii_translation}" mcp_rotation="${mcp_iii_rotation}"
-                                pp_length="${pp_iii_length}" mp_length="${mp_iii_length}" mcp_radius="${mcp_iii_radius}"
+                                pp_length="${pp_iii_length}" mp_length="${mp_iii_length}" dp_length="${dp_iii_length}"
+                                mcp_radius="${mcp_iii_radius}"
                                 pip_radius="${pip_iii_radius}" dip_radius="${dip_iii_radius}"
                                 dorsal_interossei_insertion_tf="${dorsal_interossei_iii_insertion_tf}"
@@ -288,5 +296,6 @@
                                 dp_extensor_hood_insertion_tf="${dp_iii_extensor_hood_insertion_tf}" />
                 <xacro:phalanges index="iv" mcp_translation="${mcp_iv_translation}" mcp_rotation="${mcp_iv_rotation}"
-                                pp_length="${pp_iv_length}" mp_length="${mp_iv_length}" mcp_radius="${mcp_iv_radius}"
+                                pp_length="${pp_iv_length}" mp_length="${mp_iv_length}" dp_length="${dp_iv_length}"
+                                mcp_radius="${mcp_iv_radius}"
                                 pip_radius="${pip_iv_radius}" dip_radius="${dip_iv_radius}"
                                 dorsal_interossei_insertion_tf="${dorsal_interossei_iv_insertion_tf}"
@@ -299,5 +308,5 @@
                 <xacro:phalanx_i index="i" cm_translation="${cm_i_translation}" cm_rotation="${cm_i_rotation}"
                                 centre_block_offset="${cm_i_centre_block_offset}" metacarpal_length="${metacarpal_i_length}"
-                                pp_length="${pp_i_length}" proximal_cm_radius="${proximal_cm_i_radius}"
+                                pp_length="${pp_i_length}" dp_length="${dp_i_length}" proximal_cm_radius="${proximal_cm_i_radius}"
                                 distal_cm_radius="${distal_cm_i_radius}" mcp_radius="${mcp_i_radius}" ip_radius="${ip_i_radius}"
                                 abductor_pollicis_brevis_insertion_tf="${abductor_pollicis_brevis_insertion_tf}"
@@ -317,5 +326,5 @@
                                 centre_block_offset="${cm_v_centre_block_offset}" metacarpal_length="${metacarpal_v_length}"
                                 mcp_translation="${mcp_v_translation}" mcp_rotation="${mcp_v_rotation}" pp_length="${pp_v_length}"
-                                mp_length="${mp_v_length}" proximal_cm_radius="${proximal_cm_v_radius}"
+                                mp_length="${mp_v_length}" dp_length="${dp_v_length}" proximal_cm_radius="${proximal_cm_v_radius}"
                                 distal_cm_radius="${distal_cm_v_radius}" mcp_radius="${mcp_v_radius}"
                                 pip_radius="${pip_v_radius}" dip_radius="${dip_v_radius}"

File: mujoco_env/phalanges.xml.xacro (robot description, xacro)
@@ -3,10 +3,11 @@
     <!-- Phalanges -->
     <!-- TODO: Groups -->
-    <xacro:macro name="phalanges" params="index mcp_translation mcp_rotation pp_length mp_length mcp_radius pip_radius
+    <xacro:macro name="phalanges" params="index mcp_translation mcp_rotation pp_length mp_length dp_length mcp_radius pip_radius
         dip_radius dorsal_interossei_insertion_tf palmar_interossei_insertion_tf pp_extensor_communis_insertion_tf
         flexor_superficialis_insertion_tf mp_extensor_hood_insertion_tf flexor_profundus_insertion_tf
         dp_extensor_hood_insertion_tf wrap_rgba:='0 0 1 0.2' site_rgba:='0.1 0.1 0.1 1' site_size:=0.002
         sidesite_rgba:='1 1 1 0.2' sidesite_size:=0.001 tunnelsite_size:=0.0015
-        pp_rgba:='1 0 0 1' mp_rgba:='0 1 0 1' dp_rgba:='0 0 1 1' ">
+        pp_rgba:='1 0 0 1' mp_rgba:='0 1 0 1' dp_rgba:='0 0 1 1'
+        fingertip_site_size=0.004 fingertip_site_rgba='1 0 0 0.5'">
         <body name="mcp_centre_block_${index}" pos="${mcp_translation}" euler="${mcp_rotation}">
             <joint type="hinge" axis="0 1 0" limited="true" range="-20 20" />
@@ -41,4 +42,5 @@
                         <site name="flexor_profundus_${index}_insertion" pos="${flexor_profundus_insertion_tf}" size="${site_size}" rgba="${site_rgba}"/>
                         <site name="dp_${index}_extensor_hood_insertion" pos="${dp_extensor_hood_insertion_tf}" size="${site_size}" rgba="${site_rgba}"/>
+                        <site name="fingertip_${index}" pos="0 0 ${dp_length}" size="${fingertip_site_size}" rgba="${fingertip_site_rgba}" />
                     </body>
                 </body>
@@ -47,5 +49,5 @@
     </xacro:macro>
     <xacro:macro name="phalanx_v" params="index cm_translation cm_rotation centre_block_offset metacarpal_length mcp_translation
-        mcp_rotation pp_length mp_length proximal_cm_radius distal_cm_radius mcp_radius pip_radius dip_radius dorsal_interossei_insertion_tf
+        mcp_rotation pp_length mp_length dp_length proximal_cm_radius distal_cm_radius mcp_radius pip_radius dip_radius dorsal_interossei_insertion_tf
         palmar_interossei_insertion_tf pp_extensor_communis_insertion_tf flexor_superficialis_insertion_tf
         mp_extensor_hood_insertion_tf flexor_profundus_insertion_tf dp_extensor_hood_insertion_tf
@@ -76,5 +78,6 @@
                     <site name="opponens_digiti_minimi_insertion_ii" pos="${opponens_digiti_minimi_insertion_ii_tf}" size="${tunnel_site_size}" rgba="${tunnel_site_rgba}"/>
                     <xacro:phalanges index="${index}" mcp_translation="${mcp_translation}" mcp_rotation="${mcp_rotation}"
-                                    pp_length="${pp_length}" mp_length="${mp_length}" mcp_radius="${mcp_radius}"
+                                    pp_length="${pp_length}" mp_length="${mp_length}" dp_length="${dp_length}"
+                                    mcp_radius="${mcp_radius}"
                                     pip_radius="${pip_radius}" dip_radius="${dip_radius}"
                                     dorsal_interossei_insertion_tf="${dorsal_interossei_insertion_tf}"
@@ -90,5 +93,5 @@
     </xacro:macro>
     <xacro:macro name="phalanx_i" params="index cm_translation cm_rotation centre_block_offset metacarpal_length
-        pp_length proximal_cm_radius distal_cm_radius mcp_radius ip_radius abductor_pollicis_brevis_insertion_tf
+        pp_length dp_length proximal_cm_radius distal_cm_radius mcp_radius ip_radius abductor_pollicis_brevis_insertion_tf
         abductor_pollicis_longus_insertion_tf adductor_pollicis_insertion_tf flexor_pollicis_brevis_insertion_tf
         opponens_pollicis_insertion_i_tf opponens_pollicis_insertion_ii_tf flexor_pollicis_longus_insertion_tf
@@ -97,5 +100,6 @@
         wrap_rgba:='0 0 1 0.2' pp_rgba:='1 0 0 1' dp_rgba:='0 0 1 1'
         site_size:=0.002 site_rgba:='0.1 0.1 0.1 1'
-        tunnelsite_size:=0.0015 tunnelsite_rgba:='0.5 0.5 0.5 1' sidesite_rgba:='1 1 1 0.2' ">
+        tunnelsite_size:=0.0015 tunnelsite_rgba:='0.5 0.5 0.5 1' sidesite_rgba:='1 1 1 0.2'
+        fingertip_site_size=0.004 fingertip_site_rgba='1 0 0 0.5' ">
         <body name="proximal_cm_i_centre_block" pos="${cm_translation[0]} ${cm_translation[1]} ${cm_translation[2]}" euler="${cm_rotation}">
             <joint type="hinge" axis="1 0 0" limited="true" range="-50 -10" />
@@ -136,4 +140,5 @@
                                 <site name="flexor_pollicis_longus_insertion" pos="${flexor_pollicis_longus_insertion_tf}" size="${site_size}" rgba="${site_rgba}"/>
                                 <site name="extensor_pollicis_longus_insertion" pos="${extensor_pollicis_longus_insertion_tf}" size="${site_size}" rgba="${site_rgba}"/>
+                                <site name="fingertip_${index}" pos="0 0 ${dp_length}" size="${fingertip_site_size}" rgba="${fingertip_site_rgba}" />
                             </body>
                         </body>

Commit message: RL Training Tests with RLlib and SB3

File: mujoco_env/darm_hand.xml.xacro (robot description, xacro)
@@ -183,10 +183,24 @@
     <xacro:property name="extensor_carpi_radialis_origin_tf" value="0.012 0.013 -0.065" />
     <xacro:property name="extensor_carpi_ulnaris_origin_tf" value="-0.012 0.013 -0.065" />
+    <!-- MOCAPS -->
+    <xacro:property name="fingertip_target_mocap_size" value="0.004" />
+    <xacro:property name="fingertip_target_mocap_rgba" value="1 0 0 1" />
     <!-- Tendon Origin Macro -->
     <xacro:macro name="tendon_origin" params="site_name site_tf">
         <site name="${site_name}" pos="${site_tf}" size="${origin_site_size}" rgba="${origin_site_rgba}"/>
     </xacro:macro>
+    <!-- Fingertip Mocap Target -->
+    <xacro:macro name="fingertip_target" params="hand_name name rgba:=${fingertip_target_mocap_rgba}">
+        <body name="${hand_name}_${name}" pos="0 0.25 0" mocap="true" >
+            <geom type="sphere" size="${fingertip_target_mocap_size}" rgba="${rgba}" />
+        </body>
+    </xacro:macro>
     <!-- DARM Hand -->
     <xacro:macro name="darm_hand" params="hand_name pos">
+        <xacro:fingertip_target hand_name="${hand_name}" name="fingertip_i_target" rgba="1 0 0 1" />
+        <xacro:fingertip_target hand_name="${hand_name}" name="fingertip_ii_target" rgba="0 1 0 1" />
+        <xacro:fingertip_target hand_name="${hand_name}" name="fingertip_iii_target" rgba="0 0 1 1" />
+        <xacro:fingertip_target hand_name="${hand_name}" name="fingertip_iv_target" rgba="1 1 1 1" />
+        <xacro:fingertip_target hand_name="${hand_name}" name="fingertip_v_target" rgba="0.7 0.3 0 1" />
         <body name="${hand_name}_forearm" pos="${pos}" euler="0 0 0" childclass="darm_meshes">
             <geom type="mesh" mesh="forearm_mesh" />
