Commit message: Started Gym implementation

File: mujoco_env/actuator.xml.xacro (robot description, xacro)
@@ -2,5 +2,7 @@
 <actuator xmlns:xacro="http://wiki.ros.org/xacro">
     <!-- A total of 34 muscles -->
-    <!-- Interosseis' location -->
+    <!-- IN PROGRESS: Interosseis' location -->
+    <!-- Dorsal interossei I doesn't flex regularly -->
+    <!-- Add site for flexors too -->
     <!-- Huge forces cause joint limits to be violated. Remove soft constraints -->
     <!-- Tendon damping, Joint Damping and friction -->

File: mujoco_env/darm_hand.xml.xacro (robot description, xacro)
@@ -96,4 +96,6 @@
     <xacro:property name="flexor_iii_metacarpals_tunnel_tf" value="0.007 0.0 0.051" />
     <xacro:property name="flexor_iv_metacarpals_tunnel_tf" value="-0.007 -0.005 0.051" />
+    <xacro:property name="dorsal_interossei_ii_metacarpals_tunnel_tf" value="0.034 0.002 0.074" />
+    <xacro:property name="palmar_interossei_ii_metacarpals_tunnel_tf" value="0.020 0.004 0.075" />
     <xacro:property name="extensor_communis_ii_carpals_tunnel_tf" value="0.012 0.011 0.015" />
     <xacro:property name="extensor_communis_iii_carpals_tunnel_tf" value="0.004 0.011 0.015" />
@@ -250,4 +252,6 @@
                 <site name="flexor_iii_metacarpals_tunnel" pos="${flexor_iii_metacarpals_tunnel_tf}" size="${tunnel_site_size}" rgba="${tunnel_site_rgba}"/>
                 <site name="flexor_iv_metacarpals_tunnel" pos="${flexor_iv_metacarpals_tunnel_tf}" size="${tunnel_site_size}" rgba="${tunnel_site_rgba}"/>
+                <site name="dorsal_interossei_ii_metacarpals_tunnel" pos="${dorsal_interossei_ii_metacarpals_tunnel_tf}" size="${tunnel_site_size}" rgba="${tunnel_site_rgba}"/>
+                <site name="palmar_interossei_ii_metacarpals_tunnel" pos="${palmar_interossei_ii_metacarpals_tunnel_tf}" size="${tunnel_site_size}" rgba="${tunnel_site_rgba}"/>
                 <site name="flexor_ii_carpals_tunnel" pos="${flexor_ii_carpals_tunnel_tf}" size="${tunnel_site_size}" rgba="${tunnel_site_rgba}"/>
                 <site name="flexor_iii_carpals_tunnel" pos="${flexor_iii_carpals_tunnel_tf}" size="${tunnel_site_size}" rgba="${tunnel_site_rgba}"/>

Commit message: Added Mesh files locally, referenced files from env var

File: mujoco_env/actuator.xml.xacro (robot description, xacro)
@@ -29,5 +29,5 @@
     <xacro:macro name="hand_actuators" params="hand_name">
         <!-- MACRO TO UNROLL LOOP -->
-        <xacro:macro name="make_actuators" params="tendons:=^ ctrlrange:='0 1' index:='0'">
+        <xacro:macro name="make_actuators" params="tendons:=^ ctrlrange:='0 2' index:='0'">
             <xacro:if value="${tendons}">
                 <!-- pop first item from list -->
@@ -52,15 +52,15 @@
         <xacro:property name="n_wrist" value="$(arg no_wrist)" />
         <xacro:unless value="${s_finger or n_wrist}">
-            <xacro:make_actuators tendons="${list(carpal_tendons)}" ctrlrange="0 6"/>
+            <xacro:make_actuators tendons="${list(carpal_tendons)}" ctrlrange="0 10"/>
         </xacro:unless>
         <!-- Digit II -->
-        <xacro:make_actuators tendons="${list(digitorum_tendons)}" index="ii" ctrlrange="0 1"/>
+        <xacro:make_actuators tendons="${list(digitorum_tendons)}" index="ii" ctrlrange="0 2"/>
         <!-- Pollicis, Digit III-V, Digiti Minimi Specific Tendon Actuators -->
         <xacro:unless value="$(arg single_finger)">
-            <xacro:make_actuators tendons="${list(pollicis_tendons)}" ctrlrange="0 1"/>
-            <xacro:make_actuators tendons="${list(digitorum_tendons)}" index="iii" ctrlrange="0 1"/>
-            <xacro:make_actuators tendons="${list(digitorum_tendons)}" index="iv" ctrlrange="0 1"/>
-            <xacro:make_actuators tendons="${list(digitorum_tendons)}" index="v" ctrlrange="0 1"/>
-            <xacro:make_actuators tendons="${list(digiti_minimi_specific_tendons)}" ctrlrange="0 1"/>
+            <xacro:make_actuators tendons="${list(pollicis_tendons)}" ctrlrange="0 2"/>
+            <xacro:make_actuators tendons="${list(digitorum_tendons)}" index="iii" ctrlrange="0 2"/>
+            <xacro:make_actuators tendons="${list(digitorum_tendons)}" index="iv" ctrlrange="0 2"/>
+            <xacro:make_actuators tendons="${list(digitorum_tendons)}" index="v" ctrlrange="0 2"/>
+            <xacro:make_actuators tendons="${list(digiti_minimi_specific_tendons)}" ctrlrange="0 2"/>
         </xacro:unless>
     </xacro:macro>

Commit message: Added velocity observation and increased action range to [0, 5] for single finger

File: mujoco_env/actuator.xml.xacro (robot description, xacro)
@@ -29,5 +29,5 @@
     <xacro:macro name="hand_actuators" params="hand_name">
         <!-- MACRO TO UNROLL LOOP -->
-        <xacro:macro name="make_actuators" params="tendons:=^ ctrlrange:='0 2' index:='0'">
+        <xacro:macro name="make_actuators" params="tendons:=^ ctrlrange:='0 5' index:='0'">
             <xacro:if value="${tendons}">
                 <!-- pop first item from list -->
@@ -55,12 +55,12 @@
         </xacro:unless>
         <!-- Digit II -->
-        <xacro:make_actuators tendons="${list(digitorum_tendons)}" index="ii" ctrlrange="0 2"/>
+        <xacro:make_actuators tendons="${list(digitorum_tendons)}" index="ii" ctrlrange="0 5"/>
         <!-- Pollicis, Digit III-V, Digiti Minimi Specific Tendon Actuators -->
         <xacro:unless value="$(arg single_finger)">
-            <xacro:make_actuators tendons="${list(pollicis_tendons)}" ctrlrange="0 2"/>
-            <xacro:make_actuators tendons="${list(digitorum_tendons)}" index="iii" ctrlrange="0 2"/>
-            <xacro:make_actuators tendons="${list(digitorum_tendons)}" index="iv" ctrlrange="0 2"/>
-            <xacro:make_actuators tendons="${list(digitorum_tendons)}" index="v" ctrlrange="0 2"/>
-            <xacro:make_actuators tendons="${list(digiti_minimi_specific_tendons)}" ctrlrange="0 2"/>
+            <xacro:make_actuators tendons="${list(pollicis_tendons)}" ctrlrange="0 5"/>
+            <xacro:make_actuators tendons="${list(digitorum_tendons)}" index="iii" ctrlrange="0 5"/>
+            <xacro:make_actuators tendons="${list(digitorum_tendons)}" index="iv" ctrlrange="0 5"/>
+            <xacro:make_actuators tendons="${list(digitorum_tendons)}" index="v" ctrlrange="0 5"/>
+            <xacro:make_actuators tendons="${list(digiti_minimi_specific_tendons)}" ctrlrange="0 5"/>
         </xacro:unless>
     </xacro:macro>

Commit message: Fine-Tuned Five-FIngers Env

File: mujoco_env/actuator.xml.xacro (robot description, xacro)
@@ -22,9 +22,14 @@
     'opponens_pollicis'
     ]}" />
-    <xacro:property name="digiti_minimi_specific_tendons" value="${['opponens_digiti_minimi']}" />
     <xacro:property name="digitorum_tendons" value="${[
         'dorsal_interossei', 'palmar_interossei',
-        'extensor_communis', 'flexor_profundus',
-        'flexor_superficialis']}" />
+        'flexor_profundus', 'flexor_superficialis']}" />
+    <xacro:property name="digitorum_extensor" value="${['extensor_communis']}" />
+    <xacro:property name="digiti_minimi_specific_tendons" value="${['opponens_digiti_minimi']}" />
+    <xacro:property name="carpal_tendons_max_tension" value="10" />
+    <xacro:property name="pollicis_tendons_max_tension" value="5" />
+    <xacro:property name="digitorum_tendons_max_tension" value="5" />
+    <xacro:property name="digitorum_extensor_max_tension" value="10" />
+    <xacro:property name="digiti_minimi_specific_tendons_max_tension" value="5" />
     <xacro:macro name="hand_actuators" params="hand_name">
         <!-- MACRO TO UNROLL LOOP -->
@@ -48,19 +53,26 @@
         </xacro:macro>
         <!-- Create a List of Muscles -->
-        <!-- Carpal Tendon Actuators -->
         <xacro:property name="s_finger" value="$(arg single_finger)" />
         <xacro:property name="n_wrist" value="$(arg no_wrist)" />
+        <!-- Carpal Tendon Actuators -->
         <xacro:unless value="${s_finger or n_wrist}">
-            <xacro:make_actuators tendons="${list(carpal_tendons)}" ctrlrange="0 10"/>
+            <xacro:make_actuators tendons="${list(carpal_tendons)}" ctrlrange="0 ${carpal_tendons_max_tension}"/>
+        </xacro:unless>
+        <!-- Digit I (Pollicis) Tendon Actuators -->
+        <xacro:unless value="$(arg single_finger)">
+            <xacro:make_actuators tendons="${list(pollicis_tendons)}" ctrlrange="0 ${pollicis_tendons_max_tension}"/>
         </xacro:unless>
         <!-- Digit II -->
-        <xacro:make_actuators tendons="${list(digitorum_tendons)}" index="ii" ctrlrange="0 5"/>
-        <!-- Pollicis, Digit III-V, Digiti Minimi Specific Tendon Actuators -->
+        <xacro:make_actuators tendons="${list(digitorum_tendons)}" index="ii" ctrlrange="0 ${digitorum_tendons_max_tension}"/>
+        <xacro:make_actuators tendons="${list(digitorum_extensor)}" index="ii" ctrlrange="0 ${digitorum_extensor_max_tension}"/>
+        <!-- Digit III-V, Digiti Minimi Specific Tendon Actuators -->
         <xacro:unless value="$(arg single_finger)">
-            <xacro:make_actuators tendons="${list(pollicis_tendons)}" ctrlrange="0 5"/>
-            <xacro:make_actuators tendons="${list(digitorum_tendons)}" index="iii" ctrlrange="0 5"/>
-            <xacro:make_actuators tendons="${list(digitorum_tendons)}" index="iv" ctrlrange="0 5"/>
-            <xacro:make_actuators tendons="${list(digitorum_tendons)}" index="v" ctrlrange="0 5"/>
-            <xacro:make_actuators tendons="${list(digiti_minimi_specific_tendons)}" ctrlrange="0 5"/>
+            <xacro:make_actuators tendons="${list(digitorum_tendons)}" index="iii" ctrlrange="0 ${digitorum_tendons_max_tension}"/>
+            <xacro:make_actuators tendons="${list(digitorum_extensor)}" index="iii" ctrlrange="0 ${digitorum_extensor_max_tension}"/>
+            <xacro:make_actuators tendons="${list(digitorum_tendons)}" index="iv" ctrlrange="0 ${digitorum_tendons_max_tension}"/>
+            <xacro:make_actuators tendons="${list(digitorum_extensor)}" index="iv" ctrlrange="0 ${digitorum_extensor_max_tension}"/>
+            <xacro:make_actuators tendons="${list(digitorum_tendons)}" index="v" ctrlrange="0 ${digitorum_tendons_max_tension}"/>
+            <xacro:make_actuators tendons="${list(digitorum_extensor)}" index="v" ctrlrange="0 ${digitorum_extensor_max_tension}"/>
+            <xacro:make_actuators tendons="${list(digiti_minimi_specific_tendons)}" ctrlrange="0 ${digiti_minimi_specific_tendons_max_tension}"/>
         </xacro:unless>
     </xacro:macro>

File: mujoco_env/darm_hand.xml.xacro (robot description, xacro)
@@ -202,7 +202,9 @@
     <xacro:macro name="darm_hand" params="hand_name pos">
         <!-- NOTE: Only the required mocap bodies should be exposed -->
+        <xacro:unless value="$(arg single_finger)">
+            <xacro:fingertip_target hand_name="${hand_name}" name="fingertip_i_target" rgba="1 0 0 1" />
+        </xacro:unless>
         <xacro:fingertip_target hand_name="${hand_name}" name="fingertip_ii_target" rgba="0 1 0 1" />
         <xacro:unless value="$(arg single_finger)">
-            <xacro:fingertip_target hand_name="${hand_name}" name="fingertip_i_target" rgba="1 0 0 1" />
             <xacro:fingertip_target hand_name="${hand_name}" name="fingertip_iii_target" rgba="0 0 1 1" />
             <xacro:fingertip_target hand_name="${hand_name}" name="fingertip_iv_target" rgba="1 1 1 1" />
