Commit message: Updated Mujoco xacro files to specify digits to create

File: mujoco_env/actuator.xml.xacro (robot description, xacro)
@@ -1,6 +1,10 @@
 <?xml version="1.0" encoding="UTF-8"?>
 <actuator xmlns:xacro="http://wiki.ros.org/xacro">
-    <xacro:arg name="single_finger" default="false" />
     <xacro:arg name="no_wrist" default="false" />
+    <xacro:arg name="digit_i" default="true" />
+    <xacro:arg name="digit_ii" default="true" />
+    <xacro:arg name="digit_iii" default="true" />
+    <xacro:arg name="digit_iv" default="true" />
+    <xacro:arg name="digit_v" default="true" />
     <!-- A total of 34 muscles -->
     <!-- TODO: IN PROGRESS: Interosseis' location -->
@@ -53,30 +57,36 @@
         </xacro:macro>
         <!-- Create a List of Muscles -->
-        <xacro:property name="s_finger" value="$(arg single_finger)" />
         <xacro:property name="n_wrist" value="$(arg no_wrist)" />
         <!-- Carpal Tendon Actuators -->
-        <xacro:unless value="${s_finger or n_wrist}">
+        <xacro:unless value="${n_wrist}">
             <xacro:make_actuators tendons="${list(carpal_tendons)}" ctrlrange="0 ${carpal_tendons_max_tension}"/>
         </xacro:unless>
         <!-- Digit I (Pollicis) Tendon Actuators -->
-        <xacro:unless value="$(arg single_finger)">
+        <xacro:if value="$(arg digit_i)">
             <xacro:make_actuators tendons="${list(pollicis_tendons)}" ctrlrange="0 ${pollicis_tendons_max_tension}"/>
-        </xacro:unless>
+        </xacro:if>
         <!-- Digit II -->
-        <xacro:make_actuators tendons="${list(digitorum_tendons)}" index="ii" ctrlrange="0 ${digitorum_tendons_max_tension}"/>
-        <xacro:make_actuators tendons="${list(digitorum_extensor)}" index="ii" ctrlrange="0 ${digitorum_extensor_max_tension}"/>
-        <!-- Digit III-V, Digiti Minimi Specific Tendon Actuators -->
-        <xacro:unless value="$(arg single_finger)">
+        <xacro:if value="$(arg digit_ii)">
+            <xacro:make_actuators tendons="${list(digitorum_tendons)}" index="ii" ctrlrange="0 ${digitorum_tendons_max_tension}"/>
+            <xacro:make_actuators tendons="${list(digitorum_extensor)}" index="ii" ctrlrange="0 ${digitorum_extensor_max_tension}"/>
+        </xacro:if>
+        <!-- Digit III -->
+        <xacro:if value="$(arg digit_iii)">
             <xacro:make_actuators tendons="${list(digitorum_tendons)}" index="iii" ctrlrange="0 ${digitorum_tendons_max_tension}"/>
             <xacro:make_actuators tendons="${list(digitorum_extensor)}" index="iii" ctrlrange="0 ${digitorum_extensor_max_tension}"/>
+        </xacro:if>
+        <!-- Digit IV -->
+        <xacro:if value="$(arg digit_iv)">
             <xacro:make_actuators tendons="${list(digitorum_tendons)}" index="iv" ctrlrange="0 ${digitorum_tendons_max_tension}"/>
             <xacro:make_actuators tendons="${list(digitorum_extensor)}" index="iv" ctrlrange="0 ${digitorum_extensor_max_tension}"/>
+        </xacro:if>
+        <!-- Digit V -->
+        <xacro:if value="$(arg digit_v)">
             <xacro:make_actuators tendons="${list(digitorum_tendons)}" index="v" ctrlrange="0 ${digitorum_tendons_max_tension}"/>
             <xacro:make_actuators tendons="${list(digitorum_extensor)}" index="v" ctrlrange="0 ${digitorum_extensor_max_tension}"/>
             <xacro:make_actuators tendons="${list(digiti_minimi_specific_tendons)}" ctrlrange="0 ${digiti_minimi_specific_tendons_max_tension}"/>
-        </xacro:unless>
+        </xacro:if>
     </xacro:macro>
     <xacro:hand_actuators hand_name="hand1" />
-    <!-- <xacro:hand_actuators hand_name="hand2" />
-    <xacro:hand_actuators hand_name="hand3" /> -->
+    <!-- <xacro:hand_actuators hand_name="hand2" /> -->
 </actuator>

File: mujoco_env/contact_exclusions.xml.xacro (robot description, xacro)
@@ -4,5 +4,9 @@
     <!-- TODO: Eclude contacts in Phalanx I -->
     <!-- Single Finger -->
-    <xacro:arg name="single_finger" default="false" />
+    <xacro:arg name="digit_i" default="true" />
+    <xacro:arg name="digit_ii" default="true" />
+    <xacro:arg name="digit_iii" default="true" />
+    <xacro:arg name="digit_iv" default="true" />
+    <xacro:arg name="digit_v" default="true" />
     <xacro:macro name="hand_contacts" params="hand_name">
         <!-- Carapals-Wrist -->
@@ -10,12 +14,6 @@
         <exclude body1="${hand_name}_rc_centre_block" body2="${hand_name}_forearm" />
         <exclude body1="${hand_name}_carpals_metacarpals" body2="${hand_name}_forearm" />
-        <!-- PHALANGES II -->
-        <exclude body1="${hand_name}_mcp_centre_block_ii" body2="${hand_name}_carpals_metacarpals" />
-        <exclude body1="${hand_name}_proximal_phalanx_ii" body2="${hand_name}_mcp_centre_block_ii" />
-        <exclude body1="${hand_name}_proximal_phalanx_ii" body2="${hand_name}_carpals_metacarpals" />
-        <exclude body1="${hand_name}_middle_phalanx_ii" body2="${hand_name}_proximal_phalanx_ii" />
-        <exclude body1="${hand_name}_distal_phalanx_ii" body2="${hand_name}_middle_phalanx_ii" />
-        <xacro:unless value="$(arg single_finger)">
-            <!-- PHALANGES I -->
+        <!-- PHALANGES I -->
+        <xacro:if value="$(arg digit_i)">
             <exclude body1="${hand_name}_proximal_cm_i_centre_block" body2="${hand_name}_carpals_metacarpals" />
             <exclude body1="${hand_name}_distal_cm_i_centre_block" body2="${hand_name}_proximal_cm_i_centre_block" />
@@ -26,5 +24,15 @@
             <exclude body1="${hand_name}_proximal_phalanx_i" body2="${hand_name}_metacarpal_i" />
             <exclude body1="${hand_name}_distal_phalanx_i" body2="${hand_name}_proximal_phalanx_i" />
-            <!-- PHALANGES III -->
+        </xacro:if>
+        <!-- PHALANGES II -->
+        <xacro:if value="$(arg digit_ii)">
+            <exclude body1="${hand_name}_mcp_centre_block_ii" body2="${hand_name}_carpals_metacarpals" />
+            <exclude body1="${hand_name}_proximal_phalanx_ii" body2="${hand_name}_mcp_centre_block_ii" />
+            <exclude body1="${hand_name}_proximal_phalanx_ii" body2="${hand_name}_carpals_metacarpals" />
+            <exclude body1="${hand_name}_middle_phalanx_ii" body2="${hand_name}_proximal_phalanx_ii" />
+            <exclude body1="${hand_name}_distal_phalanx_ii" body2="${hand_name}_middle_phalanx_ii" />
+        </xacro:if>
+        <!-- PHALANGES III -->
+        <xacro:if value="$(arg digit_iii)">
             <exclude body1="${hand_name}_mcp_centre_block_iii" body2="${hand_name}_carpals_metacarpals" />
             <exclude body1="${hand_name}_proximal_phalanx_iii" body2="${hand_name}_mcp_centre_block_iii" />
@@ -32,5 +40,7 @@
             <exclude body1="${hand_name}_middle_phalanx_iii" body2="${hand_name}_proximal_phalanx_iii" />
             <exclude body1="${hand_name}_distal_phalanx_iii" body2="${hand_name}_middle_phalanx_iii" />
-            <!-- PHALANGES IV -->
+        </xacro:if>
+        <!-- PHALANGES IV -->
+        <xacro:if value="$(arg digit_iv)">
             <exclude body1="${hand_name}_mcp_centre_block_iv" body2="${hand_name}_carpals_metacarpals" />
             <exclude body1="${hand_name}_proximal_phalanx_iv" body2="${hand_name}_mcp_centre_block_iv" />
@@ -38,5 +48,7 @@
             <exclude body1="${hand_name}_middle_phalanx_iv" body2="${hand_name}_proximal_phalanx_iv" />
             <exclude body1="${hand_name}_distal_phalanx_iv" body2="${hand_name}_middle_phalanx_iv" />
-            <!-- PHALANGES V -->
+        </xacro:if>
+        <!-- PHALANGES V -->
+        <xacro:if value="$(arg digit_v)">
             <exclude body1="${hand_name}_proximal_cm_v_centre_block" body2="${hand_name}_carpals_metacarpals" />
             <exclude body1="${hand_name}_distal_cm_v_centre_block" body2="${hand_name}_proximal_cm_v_centre_block" />
@@ -50,8 +62,7 @@
             <exclude body1="${hand_name}_middle_phalanx_v" body2="${hand_name}_proximal_phalanx_v" />
             <exclude body1="${hand_name}_distal_phalanx_v" body2="${hand_name}_middle_phalanx_v" />
-        </xacro:unless>
+        </xacro:if>
     </xacro:macro>
     <xacro:hand_contacts hand_name="hand1" />
-    <!-- <xacro:hand_contacts hand_name="hand2" />
-    <xacro:hand_contacts hand_name="hand3" /> -->
+    <!-- <xacro:hand_contacts hand_name="hand2" /> -->
 </contact>

File: mujoco_env/darm_hand.xml.xacro (robot description, xacro)
@@ -3,6 +3,10 @@
     <xacro:include filename="phalanges.xml.xacro" />
     <!-- Single Finger -->
-    <xacro:arg name="single_finger" default="false" />
     <xacro:arg name="no_wrist" default="false" />
+    <xacro:arg name="digit_i" default="true" />
+    <xacro:arg name="digit_ii" default="true" />
+    <xacro:arg name="digit_iii" default="true" />
+    <xacro:arg name="digit_iv" default="true" />
+    <xacro:arg name="digit_v" default="true" />
     <!-- Wrist -->
     <xacro:property name="rc_joint_tf" value="${[0, 0, 0.032]}" />
@@ -204,13 +208,24 @@
     <xacro:macro name="darm_hand" params="hand_name pos">
         <!-- NOTE: Only the required mocap bodies should be exposed -->
-        <xacro:unless value="$(arg single_finger)">
+        <!-- DIGIT I Taget MOCAP -->
+        <xacro:if value="$(arg digit_i)">
             <xacro:fingertip_target hand_name="${hand_name}" name="fingertip_i_target" rgba="1 0 0 1" />
-        </xacro:unless>
-        <xacro:fingertip_target hand_name="${hand_name}" name="fingertip_ii_target" rgba="0 1 0 1" />
-        <xacro:unless value="$(arg single_finger)">
+        </xacro:if>
+        <!-- DIGIT II Taget MOCAP -->
+        <xacro:if value="$(arg digit_ii)">
+            <xacro:fingertip_target hand_name="${hand_name}" name="fingertip_ii_target" rgba="0 1 0 1" />
+        </xacro:if>
+        <!-- DIGIT III Taget MOCAP -->
+        <xacro:if value="$(arg digit_iii)">
             <xacro:fingertip_target hand_name="${hand_name}" name="fingertip_iii_target" rgba="0 0 1 1" />
+        </xacro:if>
+        <!-- DIGIT IV Taget MOCAP -->
+        <xacro:if value="$(arg digit_iv)">
             <xacro:fingertip_target hand_name="${hand_name}" name="fingertip_iv_target" rgba="1 1 1 1" />
+        </xacro:if>
+        <!-- DIGIT V Taget MOCAP -->
+        <xacro:if value="$(arg digit_v)">
             <xacro:fingertip_target hand_name="${hand_name}" name="fingertip_v_target" rgba="0.7 0.3 0 1" />
-        </xacro:unless>
+        </xacro:if>
         <body name="${hand_name}_forearm" pos="${pos}" euler="0 0 0" childclass="darm_meshes">
             <geom type="mesh" mesh="forearm_mesh" />
@@ -309,38 +324,6 @@
                     <site name="${hand_name}_proximal_cm_i_wrap_palmar_sidesite" pos="${cm_i_translation[0]-1.2*proximal_cm_i_radius-sidesite_size} ${cm_i_translation[1]} ${cm_i_translation[2]}" size="${sidesite_size}" rgba="${sidesite_rgba}" />
                     <site name="${hand_name}_opponens_digiti_minimi_carpals_tunnel" pos="${opponens_digiti_minimi_carpals_tunnel_tf}" size="${tunnel_site_size}" rgba="${tunnel_site_rgba}" />
-                    <xacro:phalanges hand_name="${hand_name}" index="ii" mcp_translation="${mcp_ii_translation}" mcp_rotation="${mcp_ii_rotation}"
-                                    pp_length="${pp_ii_length}" mp_length="${mp_ii_length}" dp_length="${dp_ii_length}"
-                                    mcp_radius="${mcp_ii_radius}"
-                                    pip_radius="${pip_ii_radius}" dip_radius="${dip_ii_radius}"
-                                    dorsal_interossei_insertion_tf="${dorsal_interossei_ii_insertion_tf}"
-                                    palmar_interossei_insertion_tf="${palmar_interossei_ii_insertion_tf}"
-                                    pp_extensor_communis_insertion_tf="${pp_ii_extensor_communis_insertion_tf}"
-                                    flexor_superficialis_insertion_tf="${flexor_superficialis_ii_insertion_tf}"
-                                    mp_extensor_hood_insertion_tf="${mp_ii_extensor_hood_insertion_tf}"
-                                    flexor_profundus_insertion_tf="${flexor_profundus_ii_insertion_tf}"
-                                    dp_extensor_hood_insertion_tf="${dp_ii_extensor_hood_insertion_tf}" />
-                    <xacro:unless value="$(arg single_finger)">
-                        <xacro:phalanges hand_name="${hand_name}" index="iii" mcp_translation="${mcp_iii_translation}" mcp_rotation="${mcp_iii_rotation}"
-                                        pp_length="${pp_iii_length}" mp_length="${mp_iii_length}" dp_length="${dp_iii_length}"
-                                        mcp_radius="${mcp_iii_radius}"
-                                        pip_radius="${pip_iii_radius}" dip_radius="${dip_iii_radius}"
-                                        dorsal_interossei_insertion_tf="${dorsal_interossei_iii_insertion_tf}"
-                                        palmar_interossei_insertion_tf="${palmar_interossei_iii_insertion_tf}"
-                                        pp_extensor_communis_insertion_tf="${pp_iii_extensor_communis_insertion_tf}"
-                                        flexor_superficialis_insertion_tf="${flexor_superficialis_iii_insertion_tf}"
-                                        mp_extensor_hood_insertion_tf="${mp_iii_extensor_hood_insertion_tf}"
-                                        flexor_profundus_insertion_tf="${flexor_profundus_iii_insertion_tf}"
-                                        dp_extensor_hood_insertion_tf="${dp_iii_extensor_hood_insertion_tf}" />
-                        <xacro:phalanges hand_name="${hand_name}" index="iv" mcp_translation="${mcp_iv_translation}" mcp_rotation="${mcp_iv_rotation}"
-                                        pp_length="${pp_iv_length}" mp_length="${mp_iv_length}" dp_length="${dp_iv_length}"
-                                        mcp_radius="${mcp_iv_radius}"
-                                        pip_radius="${pip_iv_radius}" dip_radius="${dip_iv_radius}"
-                                        dorsal_interossei_insertion_tf="${dorsal_interossei_iv_insertion_tf}"
-                                        palmar_interossei_insertion_tf="${palmar_interossei_iv_insertion_tf}"
-                                        pp_extensor_communis_insertion_tf="${pp_iv_extensor_communis_insertion_tf}"
-                                        flexor_superficialis_insertion_tf="${flexor_superficialis_iv_insertion_tf}"
-                                        mp_extensor_hood_insertion_tf="${mp_iv_extensor_hood_insertion_tf}"
-                                        flexor_profundus_insertion_tf="${flexor_profundus_iv_insertion_tf}"
-                                        dp_extensor_hood_insertion_tf="${dp_iv_extensor_hood_insertion_tf}" />
+                    <!-- Digits I -->
+                    <xacro:if value="$(arg digit_i)">
                         <xacro:phalanx_i hand_name="${hand_name}" index="i" cm_translation="${cm_i_translation}" cm_rotation="${cm_i_rotation}"
                                         centre_block_offset="${cm_i_centre_block_offset}" metacarpal_length="${metacarpal_i_length}"
@@ -360,4 +343,49 @@
                                         pp_i_flexor_tunnel_tf="${pp_i_flexor_tunnel_tf}"
                                         pp_i_extensor_tunnel_tf="${pp_i_extensor_tunnel_tf}" />
+                    </xacro:if>
+                    <!-- Digits II -->
+                    <xacro:if value="$(arg digit_ii)">
+                        <xacro:phalanges hand_name="${hand_name}" index="ii" mcp_translation="${mcp_ii_translation}" mcp_rotation="${mcp_ii_rotation}"
+                                    pp_length="${pp_ii_length}" mp_length="${mp_ii_length}" dp_length="${dp_ii_length}"
+                                    mcp_radius="${mcp_ii_radius}"
+                                    pip_radius="${pip_ii_radius}" dip_radius="${dip_ii_radius}"
+                                    dorsal_interossei_insertion_tf="${dorsal_interossei_ii_insertion_tf}"
+                                    palmar_interossei_insertion_tf="${palmar_interossei_ii_insertion_tf}"
+                                    pp_extensor_communis_insertion_tf="${pp_ii_extensor_communis_insertion_tf}"
+                                    flexor_superficialis_insertion_tf="${flexor_superficialis_ii_insertion_tf}"
+                                    mp_extensor_hood_insertion_tf="${mp_ii_extensor_hood_insertion_tf}"
+                                    flexor_profundus_insertion_tf="${flexor_profundus_ii_insertion_tf}"
+                                    dp_extensor_hood_insertion_tf="${dp_ii_extensor_hood_insertion_tf}" />
+                    </xacro:if>
+                    <!-- Digits III -->
+                    <xacro:if value="$(arg digit_iii)">
+                        <xacro:phalanges hand_name="${hand_name}" index="iii" mcp_translation="${mcp_iii_translation}" mcp_rotation="${mcp_iii_rotation}"
+                                        pp_length="${pp_iii_length}" mp_length="${mp_iii_length}" dp_length="${dp_iii_length}"
+                                        mcp_radius="${mcp_iii_radius}"
+                                        pip_radius="${pip_iii_radius}" dip_radius="${dip_iii_radius}"
+                                        dorsal_interossei_insertion_tf="${dorsal_interossei_iii_insertion_tf}"
+                                        palmar_interossei_insertion_tf="${palmar_interossei_iii_insertion_tf}"
+                                        pp_extensor_communis_insertion_tf="${pp_iii_extensor_communis_insertion_tf}"
+                                        flexor_superficialis_insertion_tf="${flexor_superficialis_iii_insertion_tf}"
+                                        mp_extensor_hood_insertion_tf="${mp_iii_extensor_hood_insertion_tf}"
+                                        flexor_profundus_insertion_tf="${flexor_profundus_iii_insertion_tf}"
+                                        dp_extensor_hood_insertion_tf="${dp_iii_extensor_hood_insertion_tf}" />
+                    </xacro:if>
+                    <!-- Digits IV -->
+                    <xacro:if value="$(arg digit_iv)">
+                        <xacro:phalanges hand_name="${hand_name}" index="iv" mcp_translation="${mcp_iv_translation}" mcp_rotation="${mcp_iv_rotation}"
+                                        pp_length="${pp_iv_length}" mp_length="${mp_iv_length}" dp_length="${dp_iv_length}"
+                                        mcp_radius="${mcp_iv_radius}"
+                                        pip_radius="${pip_iv_radius}" dip_radius="${dip_iv_radius}"
+                                        dorsal_interossei_insertion_tf="${dorsal_interossei_iv_insertion_tf}"
+                                        palmar_interossei_insertion_tf="${palmar_interossei_iv_insertion_tf}"
+                                        pp_extensor_communis_insertion_tf="${pp_iv_extensor_communis_insertion_tf}"
+                                        flexor_superficialis_insertion_tf="${flexor_superficialis_iv_insertion_tf}"
+                                        mp_extensor_hood_insertion_tf="${mp_iv_extensor_hood_insertion_tf}"
+                                        flexor_profundus_insertion_tf="${flexor_profundus_iv_insertion_tf}"
+                                        dp_extensor_hood_insertion_tf="${dp_iv_extensor_hood_insertion_tf}" />
+                    </xacro:if>
+                    <!-- Digits V -->
+                    <xacro:if value="$(arg digit_v)">
                         <xacro:phalanx_v hand_name="${hand_name}" index="v" cm_translation="${cm_v_translation}" cm_rotation="${cm_v_rotation}"
                                         centre_block_offset="${cm_v_centre_block_offset}" metacarpal_length="${metacarpal_v_length}"
@@ -378,5 +406,5 @@
                                         opponens_digiti_minimi_insertion_ii_tf="${opponens_digiti_minimi_insertion_ii_tf}"
                                         opponens_digiti_minimi_distal_cm_v_tunnel_tf="${opponens_digiti_minimi_distal_cm_v_tunnel_tf}" />
-                    </xacro:unless>
+                    </xacro:if>
                 </body>
             </body>
@@ -384,5 +412,4 @@
     </xacro:macro>
     <xacro:darm_hand hand_name="hand1" pos="0 0 0.12" />
-    <!-- <xacro:darm_hand hand_name="hand2" pos="0.5 0 0.12" />
-    <xacro:darm_hand hand_name="hand3" pos="-0.5 0 0.12" /> -->
+    <!-- <xacro:darm_hand hand_name="hand2" pos="0.5 0 0.12" /> -->
 </worldbody>
