Commit message: Updated Mujoco xacro files to specify digits to create

File: mujoco_env/tendon.xml.xacro (robot description, xacro)
@@ -2,6 +2,10 @@
 <tendon xmlns:xacro="http://wiki.ros.org/xacro">
     <!-- TODO: Muscles with three fibres -->
-    <xacro:arg name="single_finger" default="false" />
     <xacro:arg name="no_wrist" default="false" />
+    <xacro:arg name="digit_i" default="true" />
+    <xacro:arg name="digit_ii" default="true" />
+    <xacro:arg name="digit_iii" default="true" />
+    <xacro:arg name="digit_iv" default="true" />
+    <xacro:arg name="digit_v" default="true" />
     <xacro:macro name="hand_tendons" params="hand_name">
         <xacro:macro name="phalanges_tendons" params="index hand_name">
@@ -108,14 +112,30 @@
             </spatial>
         </xacro:macro>
-        <xacro:phalanges_tendons index="ii" hand_name="${hand_name}" />
-        <!-- Digits III to V -->
-        <xacro:unless value="$(arg single_finger)">
-            <xacro:phalanges_tendons index="iii" hand_name="${hand_name}" />
-            <xacro:phalanges_tendons index="iv" hand_name="${hand_name}" />
-            <xacro:phalanges_tendons index="v" hand_name="${hand_name}" />
+        <!-- Carpals, RC Joint -->
+        <xacro:property name="n_wrist" value="$(arg no_wrist)" />
+        <xacro:unless value="${n_wrist}">
+            <spatial name="${hand_name}_flexor_carpi_radialis" width="0.0004">
+                <site site="${hand_name}_flexor_carpi_radialis_origin" />
+                <geom geom="${hand_name}_rc_joint_wrap" sidesite="${hand_name}_rc_joint_wrap_palmar_sidesite" />
+                <site site="${hand_name}_flexor_carpi_radialis_insertion" />
+            </spatial>
+            <spatial name="${hand_name}_flexor_carpi_ulnaris" width="0.0004">
+                <site site="${hand_name}_flexor_carpi_ulnaris_origin" />
+                <geom geom="${hand_name}_rc_joint_wrap" sidesite="${hand_name}_rc_joint_wrap_palmar_sidesite" />
+                <site site="${hand_name}_flexor_carpi_ulnaris_insertion" />
+            </spatial>
+            <spatial name="${hand_name}_extensor_carpi_radialis" width="0.0004">
+                <site site="${hand_name}_extensor_carpi_radialis_origin" />
+                <geom geom="${hand_name}_rc_joint_wrap" sidesite="${hand_name}_rc_joint_wrap_dorsal_sidesite" />
+                <site site="${hand_name}_extensor_carpi_radialis_insertion" />
+            </spatial>
+            <spatial name="${hand_name}_extensor_carpi_ulnaris" width="0.0004">
+                <site site="${hand_name}_extensor_carpi_ulnaris_origin" />
+                <geom geom="${hand_name}_rc_joint_wrap" sidesite="${hand_name}_rc_joint_wrap_dorsal_sidesite" />
+                <site site="${hand_name}_extensor_carpi_ulnaris_insertion" />
+            </spatial>
         </xacro:unless>
-        <!-- Pollicis and Digiti Minimi -->
-        <xacro:unless value="$(arg single_finger)">
-            <!-- Pollicis Muscles -->
+        <!-- Digits I - Pollicis Muscles -->
+        <xacro:if value="$(arg digit_i)">
             <spatial name="${hand_name}_abductor_pollicis_brevis" width="0.0004">
                 <site site="${hand_name}_abductor_pollicis_brevis_origin" />
@@ -193,5 +213,20 @@
                 <site site="${hand_name}_abductor_pollicis_longus_insertion" />
             </spatial>
-            <!-- Digiti Minimi -->
+        </xacro:if>
+        <!-- Digits II -->
+        <xacro:if value="$(arg digit_ii)">
+            <xacro:phalanges_tendons index="ii" hand_name="${hand_name}" />
+        </xacro:if>
+        <!-- Digits III -->
+        <xacro:if value="$(arg digit_iii)">
+            <xacro:phalanges_tendons index="iii" hand_name="${hand_name}" />
+        </xacro:if>
+        <!-- Digits IV -->
+        <xacro:if value="$(arg digit_iv)">
+            <xacro:phalanges_tendons index="iv" hand_name="${hand_name}" />
+        </xacro:if>
+        <!-- Digits V - Digiti Minimi-->
+        <xacro:if value="$(arg digit_v)">
+            <xacro:phalanges_tendons index="v" hand_name="${hand_name}" />
             <spatial name="${hand_name}_opponens_digiti_minimi" width="0.0004">
                 <site site="${hand_name}_opponens_digiti_minimi_origin" />
@@ -204,33 +239,7 @@
                 <site site="${hand_name}_opponens_digiti_minimi_insertion_ii" />
             </spatial>
-        </xacro:unless>
-        <!-- Carpals, RC Joint -->
-        <xacro:property name="s_finger" value="$(arg single_finger)" />
-        <xacro:property name="n_wrist" value="$(arg no_wrist)" />
-        <xacro:unless value="${s_finger or n_wrist}">
-            <spatial name="${hand_name}_flexor_carpi_radialis" width="0.0004">
-                <site site="${hand_name}_flexor_carpi_radialis_origin" />
-                <geom geom="${hand_name}_rc_joint_wrap" sidesite="${hand_name}_rc_joint_wrap_palmar_sidesite" />
-                <site site="${hand_name}_flexor_carpi_radialis_insertion" />
-            </spatial>
-            <spatial name="${hand_name}_flexor_carpi_ulnaris" width="0.0004">
-                <site site="${hand_name}_flexor_carpi_ulnaris_origin" />
-                <geom geom="${hand_name}_rc_joint_wrap" sidesite="${hand_name}_rc_joint_wrap_palmar_sidesite" />
-                <site site="${hand_name}_flexor_carpi_ulnaris_insertion" />
-            </spatial>
-            <spatial name="${hand_name}_extensor_carpi_radialis" width="0.0004">
-                <site site="${hand_name}_extensor_carpi_radialis_origin" />
-                <geom geom="${hand_name}_rc_joint_wrap" sidesite="${hand_name}_rc_joint_wrap_dorsal_sidesite" />
-                <site site="${hand_name}_extensor_carpi_radialis_insertion" />
-            </spatial>
-            <spatial name="${hand_name}_extensor_carpi_ulnaris" width="0.0004">
-                <site site="${hand_name}_extensor_carpi_ulnaris_origin" />
-                <geom geom="${hand_name}_rc_joint_wrap" sidesite="${hand_name}_rc_joint_wrap_dorsal_sidesite" />
-                <site site="${hand_name}_extensor_carpi_ulnaris_insertion" />
-            </spatial>
-        </xacro:unless>
+        </xacro:if>
     </xacro:macro>
     <xacro:hand_tendons hand_name="hand1" />
-    <!-- <xacro:hand_tendons hand_name="hand2" />
-    <xacro:hand_tendons hand_name="hand3" /> -->
+    <!-- <xacro:hand_tendons hand_name="hand2" /> -->
 </tendon>

Commit message: Position Step Servo Env

File: mujoco_env/actuator.xml.xacro (robot description, xacro)
@@ -36,5 +36,5 @@
     <xacro:property name="digitorum_extensor_max_tension" value="10" />
     <xacro:property name="digiti_minimi_specific_tendons_max_tension" value="5" />
-    <xacro:macro name="hand_actuators" params="hand_name">
+    <xacro:macro name="hand_pos_actuators" params="hand_name">
         <!-- MACRO TO UNROLL LOOP -->
         <xacro:macro name="make_actuators" params="tendons:=^ ctrlrange:='0 5' index:='0'">
@@ -43,12 +43,12 @@
                 <xacro:property name="tendon_name" value="${tendons.pop(0)}"/>
                 <xacro:unless value="${index != '0'}">
-                    <general name="${hand_name}_${tendon_name}_actuator" tendon="${hand_name}_${tendon_name}"
-                        gaintype="fixed" biastype="none" gainprm="-1" biasprm="0" ctrllimited="true" ctrlrange="${ctrlrange}"/>
+                    <position name="${hand_name}_${tendon_name}_pos_actuator" tendon="${hand_name}_${tendon_name}"
+                         kp="0" forcelimited="true" forcerange="-7 7" />
                     <!-- recursively call make_actuators -->
                     <xacro:make_actuators ctrlrange="${ctrlrange}" />
                 </xacro:unless>
                 <xacro:if value="${index != '0'}">
-                    <general name="${hand_name}_${tendon_name}_${index}_actuator" tendon="${hand_name}_${tendon_name}_${index}"
-                        gaintype="fixed" biastype="none" gainprm="-1" biasprm="0" ctrllimited="true" ctrlrange="${ctrlrange}"/>
+                    <position name="${hand_name}_${tendon_name}_${index}_pos_actuator" tendon="${hand_name}_${tendon_name}_${index}"
+                         kp="0" forcelimited="true" forcerange="-7 7" />
                     <!-- recursively call make_actuators -->
                     <xacro:make_actuators ctrlrange="${ctrlrange}" index="${index}" />
@@ -88,5 +88,58 @@
         </xacro:if>
     </xacro:macro>
-    <xacro:hand_actuators hand_name="hand1" />
+    <xacro:macro name="hand_vel_actuators" params="hand_name">
+        <!-- MACRO TO UNROLL LOOP -->
+        <xacro:macro name="make_actuators" params="tendons:=^ ctrlrange:='0 5' index:='0'">
+            <xacro:if value="${tendons}">
+                <!-- pop first item from list -->
+                <xacro:property name="tendon_name" value="${tendons.pop(0)}"/>
+                <xacro:unless value="${index != '0'}">
+                    <velocity name="${hand_name}_${tendon_name}_vel_actuator" tendon="${hand_name}_${tendon_name}"
+                         kv="0" forcelimited="true" forcerange="-7 7" />
+                    <!-- recursively call make_actuators -->
+                    <xacro:make_actuators ctrlrange="${ctrlrange}" />
+                </xacro:unless>
+                <xacro:if value="${index != '0'}">
+                    <velocity name="${hand_name}_${tendon_name}_${index}_vel_actuator" tendon="${hand_name}_${tendon_name}_${index}"
+                         kv="0" forcelimited="true" forcerange="-7 7" />
+                    <!-- recursively call make_actuators -->
+                    <xacro:make_actuators ctrlrange="${ctrlrange}" index="${index}" />
+                </xacro:if>
+            </xacro:if>
+        </xacro:macro>
+        <!-- Create a List of Muscles -->
+        <xacro:property name="n_wrist" value="$(arg no_wrist)" />
+        <!-- Carpal Tendon Actuators -->
+        <xacro:unless value="${n_wrist}">
+            <xacro:make_actuators tendons="${list(carpal_tendons)}" ctrlrange="0 ${carpal_tendons_max_tension}"/>
+        </xacro:unless>
+        <!-- Digit I (Pollicis) Tendon Actuators -->
+        <xacro:if value="$(arg digit_i)">
+            <xacro:make_actuators tendons="${list(pollicis_tendons)}" ctrlrange="0 ${pollicis_tendons_max_tension}"/>
+        </xacro:if>
+        <!-- Digit II -->
+        <xacro:if value="$(arg digit_ii)">
+            <xacro:make_actuators tendons="${list(digitorum_tendons)}" index="ii" ctrlrange="0 ${digitorum_tendons_max_tension}"/>
+            <xacro:make_actuators tendons="${list(digitorum_extensor)}" index="ii" ctrlrange="0 ${digitorum_extensor_max_tension}"/>
+        </xacro:if>
+        <!-- Digit III -->
+        <xacro:if value="$(arg digit_iii)">
+            <xacro:make_actuators tendons="${list(digitorum_tendons)}" index="iii" ctrlrange="0 ${digitorum_tendons_max_tension}"/>
+            <xacro:make_actuators tendons="${list(digitorum_extensor)}" index="iii" ctrlrange="0 ${digitorum_extensor_max_tension}"/>
+        </xacro:if>
+        <!-- Digit IV -->
+        <xacro:if value="$(arg digit_iv)">
+            <xacro:make_actuators tendons="${list(digitorum_tendons)}" index="iv" ctrlrange="0 ${digitorum_tendons_max_tension}"/>
+            <xacro:make_actuators tendons="${list(digitorum_extensor)}" index="iv" ctrlrange="0 ${digitorum_extensor_max_tension}"/>
+        </xacro:if>
+        <!-- Digit V -->
+        <xacro:if value="$(arg digit_v)">
+            <xacro:make_actuators tendons="${list(digitorum_tendons)}" index="v" ctrlrange="0 ${digitorum_tendons_max_tension}"/>
+            <xacro:make_actuators tendons="${list(digitorum_extensor)}" index="v" ctrlrange="0 ${digitorum_extensor_max_tension}"/>
+            <xacro:make_actuators tendons="${list(digiti_minimi_specific_tendons)}" ctrlrange="0 ${digiti_minimi_specific_tendons_max_tension}"/>
+        </xacro:if>
+    </xacro:macro>
+    <xacro:hand_pos_actuators hand_name="hand1" />
+    <xacro:hand_vel_actuators hand_name="hand1" />
     <!-- <xacro:hand_actuators hand_name="hand2" /> -->
 </actuator>

File: mujoco_env/darm_hand.xml.xacro (robot description, xacro)
@@ -200,7 +200,9 @@
     <xacro:macro name="fingertip_target" params="hand_name name rgba:=${fingertip_target_mocap_rgba}">
         <body name="${hand_name}_${name}" pos="0 0.25 0" mocap="true" >
-            <geom type="sphere" size="${fingertip_target_mocap_size}" rgba="${rgba}" />
+            <geom type="sphere" size="${fingertip_target_mocap_size}" rgba="${rgba}"
+                    contype="0" conaffinity="0" />
             <geom type="cylinder" size="${fingertip_target_mocap_size/2} ${3*fingertip_target_mocap_size}"
-                    pos="0 0 ${1.5*fingertip_target_mocap_size}" rgba="${rgba}" />
+                    pos="0 0 ${1.5*fingertip_target_mocap_size}" rgba="${rgba}"
+                    contype="0" conaffinity="0" />
         </body>
     </xacro:macro>
